File: _autosave-splitreus.kicad_pcb (KiCad board)
At the start: 2 copper layers, 127.5 x 99 mm, 69 parts, among them SW0 SW_PUSH, SW1 SW_PUSH, SW10 SW_PUSH, SW11 SW_PUSH, SW12 SW_PUSH, SW13 SW_PUSH, SW14 SW_PUSH, SW15 SW_PUSH, SW16 SW_PUSH, SW17 SW_PUSH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

Commit message: hot swap choc
Parts:
- U1: footprint keebio:ArduinoProMicro -> Custom Footies:nice_nano
