File: splitreus.sch (KiCad schematic (older format))
At the start: 65 parts, among them J1 TRRS, SW0 SW_PUSH, SW1 SW_PUSH, SW10 SW_PUSH, SW11 SW_PUSH, SW12 SW_PUSH, SW13 SW_PUSH, SW14 SW_PUSH, SW15 SW_PUSH, SW16 SW_PUSH, SW17 SW_PUSH, SW18 SW_PUSH, SW19 SW_PUSH, SW2 SW_PUSH, SW20 SW_PUSH, SW21 SW_PUSH, SW22 SW_PUSH, SW23 SW_PUSH, SW24 SW_PUSH, SW25 SW_PUSH, SW26 SW_PUSH, SW27 SW_PUSH, SW28 SW_PUSH, SW29 SW_PUSH, SW3 SW_PUSH, SW30 SW_PUSH, SW4 SW_PUSH, SW5 SW_PUSH, SW6 SW_PUSH, SW7 SW_PUSH, SW8 SW_PUSH, SW9 SW_PUSH, U1 ProMicro

Commit message: Lots of changes
Parts:
- added J2: LED, Connector_PinSocket_2.54mm:PinSocket_1x03_P2.54mm_Vertical, symbol Connector_Generic:Conn_01x03
- added U2, U3, U4, U5, U6: HOLE, MountingHole:MountingHole_3.2mm_M3_Pad_Via, symbol hole:HOLE
- added W1: Left, Lily58-footprint:jumper_smd_2dub, symbol jumper_smd:jumper_smd
- added W2: Right, Lily58-footprint:jumper_smd_2dub, symbol jumper_smd:jumper_smd
- D0: value DIODE_SCHOTTKY_SOT23 -> 1N4148-F; symbol Keyboard_Parts:DIODE_SCHOTTKY_SOT23 -> pspice:DIODE
- J1: footprint Lily58-footprint:MJ-4PP-9 -> Custom Footies:PJ-606-6A; symbol lily58-cache_mj-4pp-9:Lily58-cache_MJ-4PP-9 -> custom_symbols:PJ-606-6A
- RST1: footprint Connector_PinHeader_1.27mm:PinHeader_1x02_P1.27mm_Vertical -> Lily58-footprint:TACT_SWITCH_TVBP06
Connections:
- net labels added: F4

Commit message: Untested, unverified mid mount trrs
Parts:
- U2, U3, U4, U5, U6: footprint MountingHole:MountingHole_3.2mm_M3_Pad_Via -> MountingHole:MountingHole_3.2mm_M3_ISO7380_Pad
Changed lines of the file:
@@
 F 0 "U2" H 1278 6128 60  0000 L CNN
 F 1 "HOLE" H 1278 6022 60  0000 L CNN
-F 2 "MountingHole:MountingHole_3.2mm_M3_Pad_Via" H 1100 6050 60  0001 C CNN
+F 2 "MountingHole:MountingHole_3.2mm_M3_ISO7380_Pad" H 1100 6050 60  0001 C CNN
 F 3 "" H 1100 6050 60  0000 C CNN
 	1    1100 6050
@@
 F 0 "U4" H 1978 6128 60  0000 L CNN
 F 1 "HOLE" H 1978 6022 60  0000 L CNN
-F 2 "MountingHole:MountingHole_3.2mm_M3_Pad_Via" H 1800 6050 60  0001 C CNN
+F 2 "MountingHole:MountingHole_3.2mm_M3_ISO7380_Pad" H 1800 6050 60  0001 C CNN
 F 3 "" H 1800 6050 60  0000 C CNN
 	1    1800 6050
@@
 F 0 "U6" H 2828 6128 60  0000 L CNN
 F 1 "HOLE" H 2828 6022 60  0000 L CNN
-F 2 "MountingHole:MountingHole_3.2mm_M3_Pad_Via" H 2650 6050 60  0001 C CNN
+F 2 "MountingHole:MountingHole_3.2mm_M3_ISO7380_Pad" H 2650 6050 60  0001 C CNN
 F 3 "" H 2650 6050 60  0000 C CNN
 	1    2650 6050
@@
 F 0 "U3" H 1278 6728 60  0000 L CNN
 F 1 "HOLE" H 1278 6622 60  0000 L CNN
-F 2 "MountingHole:MountingHole_3.2mm_M3_Pad_Via" H 1100 6650 60  0001 C CNN
+F 2 "MountingHole:MountingHole_3.2mm_M3_ISO7380_Pad" H 1100 6650 60  0001 C CNN
 F 3 "" H 1100 6650 60  0000 C CNN
 	1    1100 6650
@@
 F 0 "U5" H 1978 6728 60  0000 L CNN
 F 1 "HOLE" H 1978 6622 60  0000 L CNN
-F 2 "MountingHole:MountingHole_3.2mm_M3_Pad_Via" H 1800 6650 60  0001 C CNN
+F 2 "MountingHole:MountingHole_3.2mm_M3_ISO7380_Pad" H 1800 6650 60  0001 C CNN
 F 3 "" H 1800 6650 60  0000 C CNN
 	1    1800 6650

Commit message: Updated to 18.05x17.05
Parts:
- removed D1, D10, D11, D12, D13, D14, D15, D16, D17, D18, D19, D2, D20, D21, D22, D23, D24, D25, D26, D27, D28, D29, D3, D30, D4, D5, D6, D7, D8, D9: DIODE_SCHOTTKY_SOT23, keebio:Diode-Hybrid-reversible, symbol Keyboard_Parts:DIODE_SCHOTTKY_SOT23
- added D1, D10, D11, D12, D13, D14, D15, D16, D17, D18, D19, D2, D20, D21, D22, D23, D24, D25, D26, D27, D28, D29, D3, D30, D4, D5, D6, D7, D8, D9: 1N4148-F, keebio:Diode-Hybrid-reversible, symbol pspice:DIODE
- J1: footprint Custom Footies:PJ-606-6A -> Lily58-footprint:TRRS_JACK_MJ4PP9; symbol custom_symbols:PJ-606-6A -> Connector:AudioJack4
- SW0, SW1, SW10, SW11, SW12, SW13, SW14, SW15, SW16, SW17, SW18, SW19, SW2, SW20, SW21, SW22, SW23, SW24, SW25, SW26, SW27, SW28, SW29, SW3, SW30, SW4, SW5, SW6, SW7, SW8, SW9: footprint Custom Footies:MX-Alps-Choc-1U-No-reversible-fixed -> keebio:Kailh-PG1350-1u-reversible-No-Clickhole
- U2, U3, U4, U5, U6: footprint MountingHole:MountingHole_3.2mm_M3_ISO7380_Pad -> MountingHole:MountingHole_2.7mm_M2.5_ISO14580_Pad

Commit message: traces
Parts:
- removed J2: LED, Connector_PinSocket_2.54mm:PinSocket_1x03_P2.54mm_Vertical, symbol Connector_Generic:Conn_01x03
Connections:
- net LED: no longer names the net of U1.16 (B1)
- no-connect marks 0 -> 5
Changed lines of the file:
@@
 	1    0    0    -1
 $EndComp
-Text GLabel 10600 2300 2    50   Input ~ 0
-LED
 $Comp
 L Connector:AudioJack4 J1
@@
 $EndComp
 $Comp
-L Connector_Generic:Conn_01x03 J2
-U 1 1 5F001DD3
-P 8800 4450
-F 0 "J2" H 8880 4492 50  0000 L CNN
-F 1 "LED" H 8880 4401 50  0000 L CNN
-F 2 "Connector_PinSocket_2.54mm:PinSocket_1x03_P2.54mm_Vertical" H 8800 4450 50  0001 C CNN
-F 3 "~" H 8800 4450 50  0001 C CNN
-	1    8800 4450
-	1    0    0    -1
-$EndComp
-Text GLabel 8600 4450 0    50   Input ~ 0
-LED
-$Comp
-L vcc:VCC #PWR0111
-U 1 1 5F0036F8
-P 8600 4350
-F 0 "#PWR0111" H 8600 4200 50  0001 C CNN
-F 1 "VCC" V 8618 4477 50  0000 L CNN
-F 2 "" H 8600 4350 50  0001 C CNN
-F 3 "" H 8600 4350 50  0001 C CNN
-	1    8600 4350
-	0    -1   -1   0
-$EndComp
-$Comp
-L gnd:GND #PWR0112
-U 1 1 5F003DD7
-P 8600 4550
-F 0 "#PWR0112" H 8600 4300 50  0001 C CNN
-F 1 "GND" V 8600 4250 50  0000 L CNN
-F 2 "" H 8600 4550 50  0001 C CNN
-F 3 "" H 8600 4550 50  0001 C CNN
-	1    8600 4550
-	0    1    1    0
-$EndComp
-$Comp
 L hole:HOLE U2
 U 1 1 5F0447E9
@@
 	1    0    0    -1
 $EndComp
+NoConn ~ 10600 2000
+NoConn ~ 10600 2100
+NoConn ~ 10600 2200
+NoConn ~ 10600 2300
+NoConn ~ 10600 1500
 $EndSCHEMATC

Commit message: Updated
Parts:
- J1: symbol Connector:AudioJack4 -> lily58-cache_mj-4pp-9:Lily58-cache_MJ-4PP-9
Connections:
- net GND: now also J1.3; no longer J1.T
- net SERIAL: now also J1.2; no longer J1.R1
- net VCC: now also J1.4; no longer J1.S
Changed lines of the file:
@@
 Text GLabel 10600 2600 2    50   Input ~ 0
 COL3
-Text GLabel 9000 3500 2    50   Input ~ 0
+Text GLabel 9000 3550 2    50   Input ~ 0
 SERIAL
 Wire Wire Line
@@
 $EndComp
 $Comp
-L Connector:AudioJack4 J1
+L lily58-cache_mj-4pp-9:Lily58-cache_MJ-4PP-9 J1
 U 1 1 5E5FAED1
-P 8800 3400
-F 0 "J1" H 8750 3450 50  0000 C CNN
-F 1 "TRRS" H 8750 3350 50  0000 C CNN
-F 2 "Lily58-footprint:TRRS_JACK_MJ4PP9" H 8800 3400 50  0001 C CNN
-F 3 "~" H 8800 3400 50  0001 C CNN
-	1    8800 3400
+P 8550 3450
+F 0 "J1" H 8500 3500 50  0000 C CNN
+F 1 "TRRS" H 8500 3400 50  0000 C CNN
+F 2 "Lily58-footprint:TRRS_JACK_MJ4PP9" H 8550 3450 50  0001 C CNN
+F 3 "~" H 8550 3450 50  0001 C CNN
+	1    8550 3450
 	1    0    0    -1
 $EndComp
@@
 L gnd:GND #PWR0107
 U 1 1 5EFFED18
-P 9000 3600
-F 0 "#PWR0107" H 9000 3350 50  0001 C CNN
-F 1 "GND" V 9000 3300 50  0000 L CNN
-F 2 "" H 9000 3600 50  0001 C CNN
-F 3 "" H 9000 3600 50  0001 C CNN
-	1    9000 3600
+P 9000 3650
+F 0 "#PWR0107" H 9000 3400 50  0001 C CNN
+F 1 "GND" V 9000 3350 50  0000 L CNN
+F 2 "" H 9000 3650 50  0001 C CNN
+F 3 "" H 9000 3650 50  0001 C CNN
+	1    9000 3650
 	0    -1   -1   0
 $EndComp

Commit message: hot swap choc
Parts:
- removed J1: TRRS, Lily58-footprint:TRRS_JACK_MJ4PP9, symbol lily58-cache_mj-4pp-9:Lily58-cache_MJ-4PP-9
- removed W1: Left, Lily58-footprint:jumper_smd_2dub, symbol jumper_smd:jumper_smd
- removed W2: Right, Lily58-footprint:jumper_smd_2dub, symbol jumper_smd:jumper_smd
- added JB: Conn_01x02, symbol Connector_Generic:Conn_01x02
- added U10, U11, U12, U13, U14, U15, U16, U17, U18, U19, U20, U21, U22, U23, U24, U25, U26, U27, U28, U29, U7, U8, U9: HOLE, symbol hole:HOLE
- D0, D1, D10, D11, D12, D13, D14, D15, D16, D17, D18, D19, D2, D20, D21, D22, D23, D24, D25, D26, D27, D28, D29, D3, D30, D4, D5, D6, D7, D8, D9: footprint keebio:Diode-Hybrid-reversible -> Custom Footies:smd_diode_reversible
- SW0, SW1, SW10, SW11, SW12, SW13, SW14, SW15, SW16, SW17, SW18, SW19, SW2, SW20, SW21, SW22, SW23, SW24, SW25, SW26, SW27, SW28, SW29, SW3, SW30, SW4, SW5, SW6, SW7, SW8, SW9: footprint keebio:Kailh-PG1350-1u-reversible-No-Clickhole -> daprice_kail_mx:Kailh_socket_PG1350_reversible
- U1: value ProMicro -> nice_nano; footprint Lily58-footprint:ProMicro_rev2 -> Custom Footies:nice_nano; symbol promicro:ProMicro -> promicro:nice_nano
- U2, U3, U4, U5, U6: footprint MountingHole:MountingHole_2.7mm_M2.5_ISO14580_Pad -> MountingHole:MountingHole_2.5mm
Connections:
- new net: JB.2 (Pin_2), U1.B+
- new net: JB.1 (Pin_1), U1.B-

Commit message: updates
Parts:
- JB1: renamed from JB; footprint (none) -> Connector_PinSocket_2.54mm:PinSocket_1x02_P2.54mm_Vertical
- U10, U11, U12, U13, U14, U15, U16, U17, U18, U19, U20, U21, U22, U23, U24, U7, U8, U9: footprint (none) -> Custom Footies:breakaway-mousebites
- U25, U26, U27, U28, U29: footprint (none) -> Custom Footies:breakaway-mousebites_half
Connections:
- net at U1.B+: no longer JB1.2 (Pin_2)
Changed lines of the file:
@@
 F 0 "U7" H 8878 6678 60  0000 L CNN
 F 1 "HOLE" H 8878 6572 60  0000 L CNN
-F 2 "" H 8700 6600 60  0000 C CNN
+F 2 "Custom Footies:breakaway-mousebites" H 8700 6600 60  0001 C CNN
 F 3 "" H 8700 6600 60  0000 C CNN
 	1    8700 6600
@@
 F 0 "U8" H 9878 6628 60  0000 L CNN
 F 1 "HOLE" H 9878 6522 60  0000 L CNN
-F 2 "" H 9700 6550 60  0000 C CNN
+F 2 "Custom Footies:breakaway-mousebites" H 9700 6550 60  0001 C CNN
 F 3 "" H 9700 6550 60  0000 C CNN
 	1    9700 6550
@@
 F 0 "U9" H 10878 6728 60  0000 L CNN
 F 1 "HOLE" H 10878 6622 60  0000 L CNN
-F 2 "" H 10700 6650 60  0000 C CNN
+F 2 "Custom Footies:breakaway-mousebites" H 10700 6650 60  0001 C CNN
 F 3 "" H 10700 6650 60  0000 C CNN
 	1    10700 6650
@@
 F 0 "U10" H 11678 6628 60  0000 L CNN
 F 1 "HOLE" H 11678 6522 60  0000 L CNN
-F 2 "" H 11500 6550 60  0000 C CNN
+F 2 "Custom Footies:breakaway-mousebites" H 11500 6550 60  0001 C CNN
 F 3 "" H 11500 6550 60  0000 C CNN
 	1    11500 6550
@@
 F 0 "U11" H 12428 6678 60  0000 L CNN
 F 1 "HOLE" H 12428 6572 60  0000 L CNN
-F 2 "" H 12250 6600 60  0000 C CNN
+F 2 "Custom Footies:breakaway-mousebites" H 12250 6600 60  0001 C CNN
 F 3 "" H 12250 6600 60  0000 C CNN
 	1    12250 6600
@@
 F 0 "U12" H 12978 6678 60  0000 L CNN
 F 1 "HOLE" H 12978 6572 60  0000 L CNN
-F 2 "" H 12800 6600 60  0000 C CNN
+F 2 "Custom Footies:breakaway-mousebites" H 12800 6600 60  0001 C CNN
 F 3 "" H 12800 6600 60  0000 C CNN
 	1    12800 6600
@@
 F 0 "U13" H 13628 6728 60  0000 L CNN
 F 1 "HOLE" H 13628 6622 60  0000 L CNN
-F 2 "" H 13450 6650 60  0000 C CNN
+F 2 "Custom Footies:breakaway-mousebites" H 13450 6650 60  0001 C CNN
 F 3 "" H 13450 6650 60  0000 C CNN
 	1    13450 6650
@@
 F 0 "U14" H 8928 7428 60  0000 L CNN
 F 1 "HOLE" H 8928 7322 60  0000 L CNN
-F 2 "" H 8750 7350 60  0000 C CNN
+F 2 "Custom Footies:breakaway-mousebites" H 8750 7350 60  0001 C CNN
 F 3 "" H 8750 7350 60  0000 C CNN
 	1    8750 7350
@@
 F 0 "U15" H 9678 7428 60  0000 L CNN
 F 1 "HOLE" H 9678 7322 60  0000 L CNN
-F 2 "" H 9500 7350 60  0000 C CNN
+F 2 "Custom Footies:breakaway-mousebites" H 9500 7350 60  0001 C CNN
 F 3 "" H 9500 7350 60  0000 C CNN
 	1    9500 7350
@@
 F 0 "U16" H 10428 7378 60  0000 L CNN
 F 1 "HOLE" H 10428 7272 60  0000 L CNN
-F 2 "" H 10250 7300 60  0000 C CNN
+F 2 "Custom Footies:breakaway-mousebites" H 10250 7300 60  0001 C CNN
 F 3 "" H 10250 7300 60  0000 C CNN
 	1    10250 7300
@@
 F 0 "U17" H 11128 7428 60  0000 L CNN
 F 1 "HOLE" H 11128 7322 60  0000 L CNN
-F 2 "" H 10950 7350 60  0000 C CNN
+F 2 "Custom Footies:breakaway-mousebites" H 10950 7350 60  0001 C CNN
 F 3 "" H 10950 7350 60  0000 C CNN
 	1    10950 7350
@@
 F 0 "U18" H 11778 7428 60  0000 L CNN
 F 1 "HOLE" H 11778 7322 60  0000 L CNN
-F 2 "" H 11600 7350 60  0000 C CNN
+F 2 "Custom Footies:breakaway-mousebites" H 11600 7350 60  0001 C CNN
 F 3 "" H 11600 7350 60  0000 C CNN
 	1    11600 7350
@@
 F 0 "U19" H 12528 7428 60  0000 L CNN
 F 1 "HOLE" H 12528 7322 60  0000 L CNN
-F 2 "" H 12350 7350 60  0000 C CNN
+F 2 "Custom Footies:breakaway-mousebites" H 12350 7350 60  0001 C CNN
 F 3 "" H 12350 7350 60  0000 C CNN
 	1    12350 7350
@@
 F 0 "U20" H 13078 7428 60  0000 L CNN
 F 1 "HOLE" H 13078 7322 60  0000 L CNN
-F 2 "" H 12900 7350 60  0000 C CNN
+F 2 "Custom Footies:breakaway-mousebites" H 12900 7350 60  0001 C CNN
 F 3 "" H 12900 7350 60  0000 C CNN
 	1    12900 7350
@@
 F 0 "U21" H 13678 7428 60  0000 L CNN
 F 1 "HOLE" H 13678 7322 60  0000 L CNN
-F 2 "" H 13500 7350 60  0000 C CNN
+F 2 "Custom Footies:breakaway-mousebites" H 13500 7350 60  0001 C CNN
 F 3 "" H 13500 7350 60  0000 C CNN
 	1    13500 7350
@@
 F 0 "U22" H 8878 7978 60  0000 L CNN
 F 1 "HOLE" H 8878 7872 60  0000 L CNN
-F 2 "" H 8700 7900 60  0000 C CNN
+F 2 "Custom Footies:breakaway-mousebites" H 8700 7900 60  0001 C CNN
 F 3 "" H 8700 7900 60  0000 C CNN
 	1    8700 7900
@@
 F 0 "U23" H 9678 7978 60  0000 L CNN
 F 1 "HOLE" H 9678 7872 60  0000 L CNN
-F 2 "" H 9500 7900 60  0000 C CNN
+F 2 "Custom Footies:breakaway-mousebites" H 9500 7900 60  0001 C CNN
 F 3 "" H 9500 7900 60  0000 C CNN
 	1    9500 7900
@@
 F 0 "U24" H 10428 7928 60  0000 L CNN
 F 1 "HOLE" H 10428 7822 60  0000 L CNN
-F 2 "" H 10250 7850 60  0000 C CNN
+F 2 "Custom Footies:breakaway-mousebites" H 10250 7850 60  0001 C CNN
 F 3 "" H 10250 7850 60  0000 C CNN
 	1    10250 7850
@@
 F 0 "U25" H 11128 7928 60  0000 L CNN
 F 1 "HOLE" H 11128 7822 60  0000 L CNN
-F 2 "" H 10950 7850 60  0000 C CNN
+F 2 "Custom Footies:breakaway-mousebites_half" H 10950 7850 60  0001 C CNN
 F 3 "" H 10950 7850 60  0000 C CNN
 	1    10950 7850
@@
 F 0 "U26" H 11778 7878 60  0000 L CNN
 F 1 "HOLE" H 11778 7772 60  0000 L CNN
-F 2 "" H 11600 7800 60  0000 C CNN
+F 2 "Custom Footies:breakaway-mousebites_half" H 11600 7800 60  0001 C CNN
 F 3 "" H 11600 7800 60  0000 C CNN
 	1    11600 7800
@@
 F 0 "U27" H 12528 7928 60  0000 L CNN
 F 1 "HOLE" H 12528 7822 60  0000 L CNN
-F 2 "" H 12350 7850 60  0000 C CNN
+F 2 "Custom Footies:breakaway-mousebites_half" H 12350 7850 60  0001 C CNN
 F 3 "" H 12350 7850 60  0000 C CNN
 	1    12350 7850
@@
 F 0 "U28" H 13128 7878 60  0000 L CNN
 F 1 "HOLE" H 13128 7772 60  0000 L CNN
-F 2 "" H 12950 7800 60  0000 C CNN
+F 2 "Custom Footies:breakaway-mousebites_half" H 12950 7800 60  0001 C CNN
 F 3 "" H 12950 7800 60  0000 C CNN
 	1    12950 7800
@@
 F 0 "U29" H 13728 7928 60  0000 L CNN
 F 1 "HOLE" H 13728 7822 60  0000 L CNN
-F 2 "" H 13550 7850 60  0000 C CNN
+F 2 "Custom Footies:breakaway-mousebites_half" H 13550 7850 60  0001 C CNN
 F 3 "" H 13550 7850 60  0000 C CNN
 	1    13550 7850
@@
 $EndComp
 $Comp
-L Connector_Generic:Conn_01x02 JB
+L Connector_Generic:Conn_01x02 JB1
 U 1 1 604F9775
 P 9850 850
-F 0 "JB" V 9814 662 50  0000 R CNN
+F 0 "JB1" V 9814 662 50  0000 R CNN
 F 1 "Conn_01x02" V 9723 662 50  0000 R CNN
-F 2 "" H 9850 850 50  0001 C CNN
+F 2 "Connector_PinSocket_2.54mm:PinSocket_1x02_P2.54mm_Vertical" H 9850 850 50  0001 C CNN
 F 3 "~" H 9850 850 50  0001 C CNN
 	1    9850 850
@@
 	9950 1050 10750 1050
 Wire Wire Line
-	10750 1050 10750 1400
-Wire Wire Line
 	10750 1400 10500 1400

Commit message: semi done
Connections:
- net COL0: now also U1.12 (B5); no longer U1.10 (E6)
- net COL1: now also U1.13 (B6); no longer U1.11 (B4)
- net COL2: now also U1.14 (B2); no longer U1.12 (B5)
- net COL3: now also U1.15 (B3); no longer U1.13 (B6)
- net COL4: now also U1.16 (B1); no longer U1.14 (B2)
- net COL5: now also U1.17 (F7); no longer U1.15 (B3)
- net ROW0: now also U1.2 (RX); no longer U1.1 (TX)
- net ROW1: now also U1.7 (D4); no longer U1.2 (RX)
- net ROW2: now also U1.8 (C6); no longer U1.5 (SCL)
- net ROW3: now also U1.9 (D7); no longer U1.7 (D4)
- net ROW4: now also U1.10 (E6); no longer U1.8 (C6)
- net ROW5: now also U1.11 (B4); no longer U1.9 (D7)
- net SERIAL: now also U1.1 (TX); no longer U1.6 (SDA)
- net at U1.B+: now also JB1.2 (Pin_2)
- new net SCL: U1.5 (SCL)
- new net SDA: U1.6 (SDA)
- no-connect marks 5 -> 3
Changed lines of the file:
@@
 Text GLabel 7400 5700 1    50   Input ~ 0
 ROW5
-Text GLabel 9200 1500 0    50   Input ~ 0
+Text GLabel 9200 1600 0    50   Input ~ 0
 ROW0
-Text GLabel 9200 1600 0    50   Input ~ 0
+Text GLabel 9200 2100 0    50   Input ~ 0
 ROW1
-Text GLabel 9200 1900 0    50   Input ~ 0
+Text GLabel 9200 2200 0    50   Input ~ 0
 ROW2
-Text GLabel 9200 2100 0    50   Input ~ 0
+Text GLabel 9200 2300 0    50   Input ~ 0
 ROW3
-Text GLabel 9200 2200 0    50   Input ~ 0
+Text GLabel 9200 2400 0    50   Input ~ 0
 ROW4
-Text GLabel 9200 2300 0    50   Input ~ 0
+Text GLabel 9200 2500 0    50   Input ~ 0
 ROW5
-Text GLabel 9200 2400 0    50   Input ~ 0
+Text GLabel 9200 2600 0    50   Input ~ 0
 COL0
-Text GLabel 9200 2500 0    50   Input ~ 0
+Text GLabel 10600 2600 2    50   Input ~ 0
 COL1
-Text GLabel 9200 2600 0    50   Input ~ 0
+Text GLabel 10600 2500 2    50   Input ~ 0
 COL2
 Text GLabel 1650 5100 3    50   Input ~ 0
@@
 Text GLabel 7550 6000 3    50   Input ~ 0
 COL5
-Text GLabel 10600 2500 2    50   Input ~ 0
+Text GLabel 10600 2300 2    50   Input ~ 0
 COL4
+Text GLabel 10600 2200 2    50   Input ~ 0
+COL5
+Text GLabel 9200 1500 0    50   Input ~ 0
+SERIAL
 Text GLabel 10600 2400 2    50   Input ~ 0
-COL5
-Text GLabel 9200 2000 0    50   Input ~ 0
-SERIAL
-Text GLabel 10600 2600 2    50   Input ~ 0
 COL3
 Wire Wire Line
@@
 $EndComp
 NoConn ~ 10600 2000
-NoConn ~ 10600 2100
-NoConn ~ 10600 2200
-NoConn ~ 10600 2300
 NoConn ~ 10600 1500
 $Comp
@@
 F 3 "" H 13550 7850 60  0000 C CNN
 	1    13550 7850
-	1    0    0    -1
-$EndComp
-$Comp
-L promicro:nice_nano U1
-U 1 1 5E46BADA
-P 9900 2250
-F 0 "U1" H 9900 3287 60  0000 C CNN
-F 1 "nice_nano" H 9900 3200 60  0000 C CNN
-F 2 "Custom Footies:nice_nano" H 10000 1200 60  0001 C CNN
-F 3 "" H 10000 1200 60  0000 C CNN
-	1    9900 2250
 	1    0    0    -1
 $EndComp
@@
 Wire Wire Line
 	10750 1400 10500 1400
+Wire Wire Line
+	10750 1050 10750 1400
+$Comp
+L promicro:nice_nano U1
+U 1 1 5E46BADA
+P 9900 2250
+F 0 "U1" H 9900 3287 60  0000 C CNN
+F 1 "nice_nano" H 9900 3200 60  0000 C CNN
+F 2 "Custom Footies:nice_nano" H 10000 1200 60  0001 C CNN
+F 3 "" H 10000 1200 60  0000 C CNN
+	1    9900 2250
+	1    0    0    -1
+$EndComp
+NoConn ~ 10600 2100
+Text GLabel 9200 1900 0    50   Input ~ 0
+SCL
+Text GLabel 9200 2000 0    50   Input ~ 0
+SDA
 $EndSCHEMATC
