File: splitreus.sch (KiCad schematic (older format))
At the start: 93 parts, among them SW0 SW_PUSH, SW1 SW_PUSH, SW10 SW_PUSH, SW11 SW_PUSH, SW12 SW_PUSH, SW13 SW_PUSH, SW14 SW_PUSH, SW15 SW_PUSH, SW16 SW_PUSH, SW17 SW_PUSH, SW18 SW_PUSH, SW19 SW_PUSH, SW2 SW_PUSH, SW20 SW_PUSH, SW21 SW_PUSH, SW22 SW_PUSH, SW23 SW_PUSH, SW24 SW_PUSH, SW25 SW_PUSH, SW26 SW_PUSH, SW27 SW_PUSH, SW28 SW_PUSH, SW29 SW_PUSH, SW3 SW_PUSH, SW30 SW_PUSH, SW4 SW_PUSH, SW5 SW_PUSH, SW6 SW_PUSH, SW7 SW_PUSH, SW8 SW_PUSH, SW9 SW_PUSH, U1 nice_nano, U10 HOLE, U11 HOLE, U12 HOLE, U13 HOLE, U14 HOLE, U15 HOLE, U16 HOLE, U17 HOLE, U18 HOLE, U19 HOLE, U2 HOLE, U20 HOLE, U21 HOLE, U22 HOLE, U23 HOLE, U24 HOLE, U25 HOLE, U26 HOLE, U27 HOLE, U28 HOLE, U29 HOLE, U3 HOLE, U4 HOLE, U5 HOLE, U6 HOLE, U7 HOLE, U8 HOLE, U9 HOLE

Commit message: design updates
Parts:
- removed RST1: RST_SWITCH, Lily58-footprint:TACT_SWITCH_TVBP06, symbol Switch:SW_Push_Open
- removed U10, U11, U12, U13, U14, U15, U16, U17, U18, U19, U20, U21, U22, U23, U24, U7, U8, U9: HOLE, Custom Footies:breakaway-mousebites, symbol hole:HOLE
- removed U25, U26, U27, U28, U29: HOLE, Custom Footies:breakaway-mousebites_half, symbol hole:HOLE

Commit message: tracies
Parts:
- removed U6: HOLE, MountingHole:MountingHole_2.5mm, symbol hole:HOLE
Changed lines of the file:
@@
-$EndComp
-$Comp
-L hole:HOLE U6
-U 1 1 5F045765
-P 2650 6050
-F 0 "U6" H 2828 6128 60  0000 L CNN
-F 1 "HOLE" H 2828 6022 60  0000 L CNN
-F 2 "MountingHole:MountingHole_2.5mm" H 2650 6050 60  0001 C CNN
-F 3 "" H 2650 6050 60  0000 C CNN
-	1    2650 6050
-	1    0    0    -1
 $EndComp
 $Comp

Commit message: aa
Parts:
- removed JB1: Conn_01x02, Connector_PinSocket_2.54mm:PinSocket_1x02_P2.54mm_Vertical, symbol Connector_Generic:Conn_01x02
- added SW91: SW_PUSH, Lily58-footprint:TACT_SWITCH_TVBP06, symbol Keyboard_Parts:SW_PUSH
Connections:
- net GND: now also SW91.2
- net RST: now also SW91.1
Changed lines of the file:
@@
 NoConn ~ 10600 2000
 NoConn ~ 10600 1500
+NoConn ~ 10600 2100
+Text GLabel 9200 1900 0    50   Input ~ 0
+SCL
+Text GLabel 9200 2000 0    50   Input ~ 0
+SDA
 $Comp
-L Connector_Generic:Conn_01x02 JB1
-U 1 1 604F9775
-P 9850 850
-F 0 "JB1" V 9814 662 50  0000 R CNN
-F 1 "Conn_01x02" V 9723 662 50  0000 R CNN
-F 2 "Connector_PinSocket_2.54mm:PinSocket_1x02_P2.54mm_Vertical" H 9850 850 50  0001 C CNN
-F 3 "~" H 9850 850 50  0001 C CNN
-	1    9850 850
+L Keyboard_Parts:SW_PUSH SW91
+U 1 1 606AC6AA
+P 11750 1700
+F 0 "SW91" H 11750 1955 50  0000 C CNN
+F 1 "SW_PUSH" H 11750 1864 50  0000 C CNN
+F 2 "Lily58-footprint:TACT_SWITCH_TVBP06" H 11750 1700 60  0001 C CNN
+F 3 "" H 11750 1700 60  0000 C CNN
+	1    11750 1700
+	1    0    0    -1
+$EndComp
+Text GLabel 11450 1700 0    50   Input ~ 0
+RST
+$Comp
+L gnd:GND #PWR0101
+U 1 1 606AE7FD
+P 12050 1700
+F 0 "#PWR0101" H 12050 1450 50  0001 C CNN
+F 1 "GND" V 12050 1400 50  0000 L CNN
+F 2 "" H 12050 1700 50  0001 C CNN
+F 3 "" H 12050 1700 50  0001 C CNN
+	1    12050 1700
 	0    -1   -1   0
 $EndComp
-Wire Wire Line
-	9300 1400 9000 1400
-Wire Wire Line
-	9000 1400 9000 1050
-Wire Wire Line
-	9000 1050 9850 1050
-Wire Wire Line
-	9950 1050 10750 1050
-Wire Wire Line
-	10750 1400 10500 1400
-Wire Wire Line
-	10750 1050 10750 1400
 $Comp
 L promicro:nice_nano U1
@@
 	1    0    0    -1
 $EndComp
-NoConn ~ 10600 2100
-Text GLabel 9200 1900 0    50   Input ~ 0
-SCL
-Text GLabel 9200 2000 0    50   Input ~ 0
-SDA
 $EndSCHEMATC

Commit message: changes
Parts:
- removed D0, D1, D10, D15, D2, D20, D25, D3, D4, D5: 1N4148-F, Custom Footies:smd_diode_reversible, symbol pspice:DIODE
- removed SW0, SW1, SW10, SW15, SW2, SW20, SW25, SW3, SW4, SW5: SW_PUSH, daprice_kail_mx:Kailh_socket_PG1350_reversible, symbol Keyboard_Parts:SW_PUSH
- added J3: Conn_01x04, Lily58-footprint:TRRS_JACK_MJ4PP9, symbol Connector_Generic:Conn_01x04
- U1: symbol promicro:nice_nano -> Keyboard_Parts:Pro_Micro
Connections:
- net GND: now also J3.4 (Pin_4)
- net SCL: now also J3.1 (Pin_1)
- net SDA: now also J3.2 (Pin_2)
- net VCC: now also J3.3 (Pin_3)

Commit message: change
Parts:
- added U6, U7, U8, U9: HOLE, MountingHole:MountingHole_2.2mm_M2, symbol hole:HOLE
- J3: footprint Lily58-footprint:TRRS_JACK_MJ4PP9 -> Connector:FanPinHeader_1x04_P2.54mm_Vertical
- U2, U3, U4, U5: footprint MountingHole:MountingHole_2.5mm -> MountingHole:MountingHole_2.2mm_M2
Changed lines of the file:
@@
 F 0 "U2" H 1278 6128 60  0000 L CNN
 F 1 "HOLE" H 1278 6022 60  0000 L CNN
-F 2 "MountingHole:MountingHole_2.5mm" H 1100 6050 60  0001 C CNN
+F 2 "MountingHole:MountingHole_2.2mm_M2" H 1100 6050 60  0001 C CNN
 F 3 "" H 1100 6050 60  0000 C CNN
 	1    1100 6050
@@
 F 0 "U4" H 1978 6128 60  0000 L CNN
 F 1 "HOLE" H 1978 6022 60  0000 L CNN
-F 2 "MountingHole:MountingHole_2.5mm" H 1800 6050 60  0001 C CNN
+F 2 "MountingHole:MountingHole_2.2mm_M2" H 1800 6050 60  0001 C CNN
 F 3 "" H 1800 6050 60  0000 C CNN
 	1    1800 6050
@@
 F 0 "U3" H 1278 6728 60  0000 L CNN
 F 1 "HOLE" H 1278 6622 60  0000 L CNN
-F 2 "MountingHole:MountingHole_2.5mm" H 1100 6650 60  0001 C CNN
+F 2 "MountingHole:MountingHole_2.2mm_M2" H 1100 6650 60  0001 C CNN
 F 3 "" H 1100 6650 60  0000 C CNN
 	1    1100 6650
@@
 F 0 "U5" H 1978 6728 60  0000 L CNN
 F 1 "HOLE" H 1978 6622 60  0000 L CNN
-F 2 "MountingHole:MountingHole_2.5mm" H 1800 6650 60  0001 C CNN
+F 2 "MountingHole:MountingHole_2.2mm_M2" H 1800 6650 60  0001 C CNN
 F 3 "" H 1800 6650 60  0000 C CNN
 	1    1800 6650
@@
 F 0 "J3" H 10530 3592 50  0000 L CNN
 F 1 "Conn_01x04" H 10530 3501 50  0000 L CNN
-F 2 "Lily58-footprint:TRRS_JACK_MJ4PP9" H 10450 3600 50  0001 C CNN
+F 2 "Connector:FanPinHeader_1x04_P2.54mm_Vertical" H 10450 3600 50  0001 C CNN
 F 3 "~" H 10450 3600 50  0001 C CNN
 	1    10450 3600
@@
 Text GLabel 2600 2100 1    50   Input ~ 0
 ROW1
+$Comp
+L hole:HOLE U6
+U 1 1 60C66EBC
+P 2550 6050
+F 0 "U6" H 2728 6128 60  0000 L CNN
+F 1 "HOLE" H 2728 6022 60  0000 L CNN
+F 2 "MountingHole:MountingHole_2.2mm_M2" H 2550 6050 60  0001 C CNN
+F 3 "" H 2550 6050 60  0000 C CNN
+	1    2550 6050
+	1    0    0    -1
+$EndComp
+$Comp
+L hole:HOLE U8
+U 1 1 60C66EC2
+P 3250 6050
+F 0 "U8" H 3428 6128 60  0000 L CNN
+F 1 "HOLE" H 3428 6022 60  0000 L CNN
+F 2 "MountingHole:MountingHole_2.2mm_M2" H 3250 6050 60  0001 C CNN
+F 3 "" H 3250 6050 60  0000 C CNN
+	1    3250 6050
+	1    0    0    -1
+$EndComp
+$Comp
+L hole:HOLE U7
+U 1 1 60C66EC8
+P 2550 6650
+F 0 "U7" H 2728 6728 60  0000 L CNN
+F 1 "HOLE" H 2728 6622 60  0000 L CNN
+F 2 "MountingHole:MountingHole_2.2mm_M2" H 2550 6650 60  0001 C CNN
+F 3 "" H 2550 6650 60  0000 C CNN
+	1    2550 6650
+	1    0    0    -1
+$EndComp
+$Comp
+L hole:HOLE U9
+U 1 1 60C66ECE
+P 3250 6650
+F 0 "U9" H 3428 6728 60  0000 L CNN
+F 1 "HOLE" H 3428 6622 60  0000 L CNN
+F 2 "MountingHole:MountingHole_2.2mm_M2" H 3250 6650 60  0001 C CNN
+F 3 "" H 3250 6650 60  0000 C CNN
+	1    3250 6650
+	1    0    0    -1
+$EndComp
 $EndSCHEMATC

Commit message: fin?
Parts:
- removed J3: Conn_01x04, Connector:FanPinHeader_1x04_P2.54mm_Vertical, symbol Connector_Generic:Conn_01x04
- removed U7: HOLE, MountingHole:MountingHole_2.2mm_M2, symbol hole:HOLE
- SW11, SW12, SW13, SW14, SW16, SW17, SW18, SW19, SW21, SW22, SW23, SW24, SW26, SW27, SW28, SW29, SW30, SW6, SW7, SW8, SW9: footprint daprice_kail_mx:Kailh_socket_PG1350_reversible -> Custom Footies:choc_hs_reversible
- U2, U3, U4, U5, U6, U8, U9: footprint MountingHole:MountingHole_2.2mm_M2 -> Custom Footies:MountingHole_2.2mm_M2
Changed lines of the file:
@@
 F 0 "SW6" H 2300 2355 50  0000 C CNN
 F 1 "SW_PUSH" H 2300 2264 50  0000 C CNN
-F 2 "daprice_kail_mx:Kailh_socket_PG1350_reversible" H 2300 2100 60  0001 C CNN
+F 2 "Custom Footies:choc_hs_reversible" H 2300 2100 60  0001 C CNN
 F 3 "" H 2300 2100 60  0000 C CNN
 	1    2300 2100
@@
 F 0 "SW7" H 2300 3255 50  0000 C CNN
 F 1 "SW_PUSH" H 2300 3164 50  0000 C CNN
-F 2 "daprice_kail_mx:Kailh_socket_PG1350_reversible" H 2300 3000 60  0001 C CNN
+F 2 "Custom Footies:choc_hs_reversible" H 2300 3000 60  0001 C CNN
 F 3 "" H 2300 3000 60  0000 C CNN
 	1    2300 3000
@@
 F 0 "SW8" H 2300 4155 50  0000 C CNN
 F 1 "SW_PUSH" H 2300 4064 50  0000 C CNN
-F 2 "daprice_kail_mx:Kailh_socket_PG1350_reversible" H 2300 3900 60  0001 C CNN
+F 2 "Custom Footies:choc_hs_reversible" H 2300 3900 60  0001 C CNN
 F 3 "" H 2300 3900 60  0000 C CNN
 	1    2300 3900
@@
 F 0 "SW9" H 2300 5055 50  0000 C CNN
 F 1 "SW_PUSH" H 2300 4964 50  0000 C CNN
-F 2 "daprice_kail_mx:Kailh_socket_PG1350_reversible" H 2300 4800 60  0001 C CNN
+F 2 "Custom Footies:choc_hs_reversible" H 2300 4800 60  0001 C CNN
 F 3 "" H 2300 4800 60  0000 C CNN
 	1    2300 4800
@@
 F 0 "SW11" H 3450 2355 50  0000 C CNN
 F 1 "SW_PUSH" H 3450 2264 50  0000 C CNN
-F 2 "daprice_kail_mx:Kailh_socket_PG1350_reversible" H 3450 2100 60  0001 C CNN
+F 2 "Custom Footies:choc_hs_reversible" H 3450 2100 60  0001 C CNN
 F 3 "" H 3450 2100 60  0000 C CNN
 	1    3450 2100
@@
 F 0 "SW12" H 3450 3255 50  0000 C CNN
 F 1 "SW_PUSH" H 3450 3164 50  0000 C CNN
-F 2 "daprice_kail_mx:Kailh_socket_PG1350_reversible" H 3450 3000 60  0001 C CNN
+F 2 "Custom Footies:choc_hs_reversible" H 3450 3000 60  0001 C CNN
 F 3 "" H 3450 3000 60  0000 C CNN
 	1    3450 3000
@@
 F 0 "SW13" H 3450 4155 50  0000 C CNN
 F 1 "SW_PUSH" H 3450 4064 50  0000 C CNN
-F 2 "daprice_kail_mx:Kailh_socket_PG1350_reversible" H 3450 3900 60  0001 C CNN
+F 2 "Custom Footies:choc_hs_reversible" H 3450 3900 60  0001 C CNN
 F 3 "" H 3450 3900 60  0000 C CNN
 	1    3450 3900
@@
 F 0 "SW14" H 3450 5055 50  0000 C CNN
 F 1 "SW_PUSH" H 3450 4964 50  0000 C CNN
-F 2 "daprice_kail_mx:Kailh_socket_PG1350_reversible" H 3450 4800 60  0001 C CNN
+F 2 "Custom Footies:choc_hs_reversible" H 3450 4800 60  0001 C CNN
 F 3 "" H 3450 4800 60  0000 C CNN
 	1    3450 4800
@@
 F 0 "SW16" H 4600 2355 50  0000 C CNN
 F 1 "SW_PUSH" H 4600 2264 50  0000 C CNN
-F 2 "daprice_kail_mx:Kailh_socket_PG1350_reversible" H 4600 2100 60  0001 C CNN
+F 2 "Custom Footies:choc_hs_reversible" H 4600 2100 60  0001 C CNN
 F 3 "" H 4600 2100 60  0000 C CNN
 	1    4600 2100
@@
 F 0 "SW17" H 4600 3255 50  0000 C CNN
 F 1 "SW_PUSH" H 4600 3164 50  0000 C CNN
-F 2 "daprice_kail_mx:Kailh_socket_PG1350_reversible" H 4600 3000 60  0001 C CNN
+F 2 "Custom Footies:choc_hs_reversible" H 4600 3000 60  0001 C CNN
 F 3 "" H 4600 3000 60  0000 C CNN
 	1    4600 3000
@@
 F 0 "SW18" H 4600 4155 50  0000 C CNN
 F 1 "SW_PUSH" H 4600 4064 50  0000 C CNN
-F 2 "daprice_kail_mx:Kailh_socket_PG1350_reversible" H 4600 3900 60  0001 C CNN
+F 2 "Custom Footies:choc_hs_reversible" H 4600 3900 60  0001 C CNN
 F 3 "" H 4600 3900 60  0000 C CNN
 	1    4600 3900
@@
 F 0 "SW19" H 4600 5055 50  0000 C CNN
 F 1 "SW_PUSH" H 4600 4964 50  0000 C CNN
-F 2 "daprice_kail_mx:Kailh_socket_PG1350_reversible" H 4600 4800 60  0001 C CNN
+F 2 "Custom Footies:choc_hs_reversible" H 4600 4800 60  0001 C CNN
 F 3 "" H 4600 4800 60  0000 C CNN
 	1    4600 4800
@@
 F 0 "SW21" H 5850 2355 50  0000 C CNN
 F 1 "SW_PUSH" H 5850 2264 50  0000 C CNN
-F 2 "daprice_kail_mx:Kailh_socket_PG1350_reversible" H 5850 2100 60  0001 C CNN
+F 2 "Custom Footies:choc_hs_reversible" H 5850 2100 60  0001 C CNN
 F 3 "" H 5850 2100 60  0000 C CNN
 	1    5850 2100
@@
 F 0 "SW22" H 5850 3255 50  0000 C CNN
 F 1 "SW_PUSH" H 5850 3164 50  0000 C CNN
-F 2 "daprice_kail_mx:Kailh_socket_PG1350_reversible" H 5850 3000 60  0001 C CNN
+F 2 "Custom Footies:choc_hs_reversible" H 5850 3000 60  0001 C CNN
 F 3 "" H 5850 3000 60  0000 C CNN
 	1    5850 3000
@@
 F 0 "SW23" H 5850 4155 50  0000 C CNN
 F 1 "SW_PUSH" H 5850 4064 50  0000 C CNN
-F 2 "daprice_kail_mx:Kailh_socket_PG1350_reversible" H 5850 3900 60  0001 C CNN
+F 2 "Custom Footies:choc_hs_reversible" H 5850 3900 60  0001 C CNN
 F 3 "" H 5850 3900 60  0000 C CNN
 	1    5850 3900
@@
 F 0 "SW24" H 5850 5055 50  0000 C CNN
 F 1 "SW_PUSH" H 5850 4964 50  0000 C CNN
-F 2 "daprice_kail_mx:Kailh_socket_PG1350_reversible" H 5850 4800 60  0001 C CNN
+F 2 "Custom Footies:choc_hs_reversible" H 5850 4800 60  0001 C CNN
 F 3 "" H 5850 4800 60  0000 C CNN
 	1    5850 4800
@@
 F 0 "SW26" H 7100 2355 50  0000 C CNN
 F 1 "SW_PUSH" H 7100 2264 50  0000 C CNN
-F 2 "daprice_kail_mx:Kailh_socket_PG1350_reversible" H 7100 2100 60  0001 C CNN
+F 2 "Custom Footies:choc_hs_reversible" H 7100 2100 60  0001 C CNN
 F 3 "" H 7100 2100 60  0000 C CNN
 	1    7100 2100
@@
 F 0 "SW27" H 7100 3255 50  0000 C CNN
 F 1 "SW_PUSH" H 7100 3164 50  0000 C CNN
-F 2 "daprice_kail_mx:Kailh_socket_PG1350_reversible" H 7100 3000 60  0001 C CNN
+F 2 "Custom Footies:choc_hs_reversible" H 7100 3000 60  0001 C CNN
 F 3 "" H 7100 3000 60  0000 C CNN
 	1    7100 3000
@@
 F 0 "SW28" H 7100 4155 50  0000 C CNN
 F 1 "SW_PUSH" H 7100 4064 50  0000 C CNN
-F 2 "daprice_kail_mx:Kailh_socket_PG1350_reversible" H 7100 3900 60  0001 C CNN
+F 2 "Custom Footies:choc_hs_reversible" H 7100 3900 60  0001 C CNN
 F 3 "" H 7100 3900 60  0000 C CNN
 	1    7100 3900
@@
 F 0 "SW29" H 7100 5055 50  0000 C CNN
 F 1 "SW_PUSH" H 7100 4964 50  0000 C CNN
-F 2 "daprice_kail_mx:Kailh_socket_PG1350_reversible" H 7100 4800 60  0001 C CNN
+F 2 "Custom Footies:choc_hs_reversible" H 7100 4800 60  0001 C CNN
 F 3 "" H 7100 4800 60  0000 C CNN
 	1    7100 4800
@@
 F 0 "SW30" H 7100 5955 50  0000 C CNN
 F 1 "SW_PUSH" H 7100 5864 50  0000 C CNN
-F 2 "daprice_kail_mx:Kailh_socket_PG1350_reversible" H 7100 5700 60  0001 C CNN
+F 2 "Custom Footies:choc_hs_reversible" H 7100 5700 60  0001 C CNN
 F 3 "" H 7100 5700 60  0000 C CNN
 	1    7100 5700
@@
 F 0 "U2" H 1278 6128 60  0000 L CNN
 F 1 "HOLE" H 1278 6022 60  0000 L CNN
-F 2 "MountingHole:MountingHole_2.2mm_M2" H 1100 6050 60  0001 C CNN
+F 2 "Custom Footies:MountingHole_2.2mm_M2" H 1100 6050 60  0001 C CNN
 F 3 "" H 1100 6050 60  0000 C CNN
 	1    1100 6050
@@
 F 0 "U4" H 1978 6128 60  0000 L CNN
 F 1 "HOLE" H 1978 6022 60  0000 L CNN
-F 2 "MountingHole:MountingHole_2.2mm_M2" H 1800 6050 60  0001 C CNN
+F 2 "Custom Footies:MountingHole_2.2mm_M2" H 1800 6050 60  0001 C CNN
 F 3 "" H 1800 6050 60  0000 C CNN
 	1    1800 6050
@@
 F 0 "U3" H 1278 6728 60  0000 L CNN
 F 1 "HOLE" H 1278 6622 60  0000 L CNN
-F 2 "MountingHole:MountingHole_2.2mm_M2" H 1100 6650 60  0001 C CNN
+F 2 "Custom Footies:MountingHole_2.2mm_M2" H 1100 6650 60  0001 C CNN
 F 3 "" H 1100 6650 60  0000 C CNN
 	1    1100 6650
@@
 F 0 "U5" H 1978 6728 60  0000 L CNN
 F 1 "HOLE" H 1978 6622 60  0000 L CNN
-F 2 "MountingHole:MountingHole_2.2mm_M2" H 1800 6650 60  0001 C CNN
+F 2 "Custom Footies:MountingHole_2.2mm_M2" H 1800 6650 60  0001 C CNN
 F 3 "" H 1800 6650 60  0000 C CNN
 	1    1800 6650
@@
 	1    0    0    -1
 $EndComp
-Text GLabel 10250 3500 0    50   Input ~ 0
-SCL
-$Comp
-L gnd:GND #PWR0102
-U 1 1 60C28C17
-P 10250 3800
-F 0 "#PWR0102" H 10250 3550 50  0001 C CNN
-F 1 "GND" H 10250 3650 50  0000 C CNN
-F 2 "" H 10250 3800 50  0001 C CNN
-F 3 "" H 10250 3800 50  0001 C CNN
-	1    10250 3800
-	1    0    0    -1
-$EndComp
-$Comp
-L vcc:VCC #PWR0107
-U 1 1 60C29E2D
-P 10250 3700
-F 0 "#PWR0107" H 10250 3550 50  0001 C CNN
-F 1 "VCC" V 10200 3850 50  0000 L CNN
-F 2 "" H 10250 3700 50  0001 C CNN
-F 3 "" H 10250 3700 50  0001 C CNN
-	1    10250 3700
-	0    -1   -1   0
-$EndComp
-$Comp
-L Connector_Generic:Conn_01x04 J3
-U 1 1 60C3C374
-P 10450 3600
-F 0 "J3" H 10530 3592 50  0000 L CNN
-F 1 "Conn_01x04" H 10530 3501 50  0000 L CNN
-F 2 "Connector:FanPinHeader_1x04_P2.54mm_Vertical" H 10450 3600 50  0001 C CNN
-F 3 "~" H 10450 3600 50  0001 C CNN
-	1    10450 3600
-	1    0    0    -1
-$EndComp
-Text GLabel 10250 3600 0    50   Input ~ 0
-SDA
 Text GLabel 7400 2100 1    50   Input ~ 0
 ROW1
@@
 F 0 "U6" H 2728 6128 60  0000 L CNN
 F 1 "HOLE" H 2728 6022 60  0000 L CNN
-F 2 "MountingHole:MountingHole_2.2mm_M2" H 2550 6050 60  0001 C CNN
+F 2 "Custom Footies:MountingHole_2.2mm_M2" H 2550 6050 60  0001 C CNN
 F 3 "" H 2550 6050 60  0000 C CNN
 	1    2550 6050
@@
 F 0 "U8" H 3428 6128 60  0000 L CNN
 F 1 "HOLE" H 3428 6022 60  0000 L CNN
-F 2 "MountingHole:MountingHole_2.2mm_M2" H 3250 6050 60  0001 C CNN
+F 2 "Custom Footies:MountingHole_2.2mm_M2" H 3250 6050 60  0001 C CNN
 F 3 "" H 3250 6050 60  0000 C CNN
 	1    3250 6050
-	1    0    0    -1
-$EndComp
-$Comp
-L hole:HOLE U7
-U 1 1 60C66EC8
-P 2550 6650
-F 0 "U7" H 2728 6728 60  0000 L CNN
-F 1 "HOLE" H 2728 6622 60  0000 L CNN
-F 2 "MountingHole:MountingHole_2.2mm_M2" H 2550 6650 60  0001 C CNN
-F 3 "" H 2550 6650 60  0000 C CNN
-	1    2550 6650
 	1    0    0    -1
 $EndComp
@@
 F 0 "U9" H 3428 6728 60  0000 L CNN
 F 1 "HOLE" H 3428 6622 60  0000 L CNN
-F 2 "MountingHole:MountingHole_2.2mm_M2" H 3250 6650 60  0001 C CNN
+F 2 "Custom Footies:MountingHole_2.2mm_M2" H 3250 6650 60  0001 C CNN
 F 3 "" H 3250 6650 60  0000 C CNN
 	1    3250 6650
