File: splitreus.sch (KiCad schematic (older format))
At the start: 65 parts, among them J1 TRRS, SW0 SW_PUSH, SW1 SW_PUSH, SW10 SW_PUSH, SW11 SW_PUSH, SW12 SW_PUSH, SW13 SW_PUSH, SW14 SW_PUSH, SW15 SW_PUSH, SW16 SW_PUSH, SW17 SW_PUSH, SW18 SW_PUSH, SW19 SW_PUSH, SW2 SW_PUSH, SW20 SW_PUSH, SW21 SW_PUSH, SW22 SW_PUSH, SW23 SW_PUSH, SW24 SW_PUSH, SW25 SW_PUSH, SW26 SW_PUSH, SW27 SW_PUSH, SW28 SW_PUSH, SW29 SW_PUSH, SW3 SW_PUSH, SW30 SW_PUSH, SW4 SW_PUSH, SW5 SW_PUSH, SW6 SW_PUSH, SW7 SW_PUSH, SW8 SW_PUSH, SW9 SW_PUSH, U1 ProMicro

Commit message: a lot
Parts:
- D0, D1, D10, D11, D12, D13, D14, D15, D16, D17, D18, D19, D2, D20, D21, D22, D23, D24, D25, D26, D27, D28, D29, D3, D30, D4, D5, D6, D7, D8, D9: value DIODE_SCHOTTKY_SOT23 -> 1N4148; footprint keebio:Diode-Hybrid-reversible -> Custom Footies:Diode-Hybrid-reversible; symbol Keyboard_Parts:DIODE_SCHOTTKY_SOT23 -> pspice:DIODE
- RST1: footprint Connector_PinHeader_1.27mm:PinHeader_1x02_P1.27mm_Vertical -> Lily58-footprint:TACT_SWITCH_TVBP06
- SW0, SW1, SW10, SW11, SW12, SW13, SW14, SW15, SW16, SW17, SW18, SW19, SW2, SW20, SW21, SW22, SW23, SW24, SW25, SW26, SW27, SW28, SW29, SW3, SW30, SW4, SW5, SW6, SW7, SW8, SW9: footprint Custom Footies:MX-Alps-Choc-1U-No-reversible-fixed -> daprice_kail_mx:Kailh_socket_MX_reversible
- U1: footprint Lily58-footprint:ProMicro_rev2 -> Custom Footies:nice_nano
Connections:
- wire segments 149 -> 157
- no-connect marks 0 -> 3

Commit message: traces
Parts:
- added J2: battery, Connector_PinSocket_2.54mm:PinSocket_1x02_P2.54mm_Vertical, symbol Connector:Conn_01x02_Male
- SW0, SW1, SW10, SW11, SW12, SW13, SW14, SW15, SW16, SW17, SW18, SW19, SW2, SW20, SW21, SW22, SW23, SW24, SW25, SW26, SW27, SW28, SW29, SW3, SW30, SW4, SW5, SW6, SW7, SW8, SW9: footprint daprice_kail_mx:Kailh_socket_MX_reversible -> Custom Footies:Kailh_socket_MX_reversible_fix
- U1: symbol promicro:ProMicro -> promicro:nice_nano
Connections:
- net labels added: B+, B-

Commit message: traces routed
Parts:
- added D0, D1, D10, D11, D12, D13, D14, D15, D16, D17, D18, D19, D2, D20, D21, D22, D23, D24, D25, D26, D27, D28, D29, D3, D30, D4, D5, D6, D7, D8, D9: SK6812MINI, LED_SMD:LED_SK6812MINI_PLCC4_3.5x3.5mm_P1.75mm, symbol LED:SK6812MINI
Connections:
- net GND: now also D0.2 (VSS), D1.2 (VSS), D10.2 (VSS), D11.2 (VSS), D12.2 (VSS), D13.2 (VSS), D14.2 (VSS), D15.2 (VSS), D16.2 (VSS), D17.2 (VSS), D18.2 (VSS), D19.2 (VSS), D2.2 (VSS), D20.2 (VSS), D21.2 (VSS), D22.2 (VSS), D23.2 (VSS), D24.2 (VSS), D25.2 (VSS), D26.2 (VSS), D27.2 (VSS), D28.2 (VSS), D29.2 (VSS), D3.2 (VSS), D30.2 (VSS), D4.2 (VSS), D5.2 (VSS), D6.2 (VSS), D7.2 (VSS), D8.2 (VSS), D9.2 (VSS)
- net LED: now also D4.3 (DIN)
- net VCC: now also D0.4 (VDD), D1.4 (VDD), D10.4 (VDD), D11.4 (VDD), D12.4 (VDD), D13.4 (VDD), D14.4 (VDD), D15.4 (VDD), D16.4 (VDD), D17.4 (VDD), D18.4 (VDD), D19.4 (VDD), D2.4 (VDD), D20.4 (VDD), D21.4 (VDD), D22.4 (VDD), D23.4 (VDD), D24.4 (VDD), D25.4 (VDD), D26.4 (VDD), D27.4 (VDD), D28.4 (VDD), D29.4 (VDD), D3.4 (VDD), D30.4 (VDD), D4.4 (VDD), D5.4 (VDD), D6.4 (VDD), D7.4 (VDD), D8.4 (VDD), D9.4 (VDD)
- net to_right: now reaches J1.1
- net to_right: now also D30.1 (DOUT)
- new net: D3.3 (DIN), D4.1 (DOUT)
- new net: D2.3 (DIN), D3.1 (DOUT)
- new net: D1.3 (DIN), D2.1 (DOUT)
- new net: D0.3 (DIN), D1.1 (DOUT)
- new net: D0.1 (DOUT), D9.3 (DIN)
- new net: D8.3 (DIN), D9.1 (DOUT)
- new net: D7.3 (DIN), D8.1 (DOUT)
- new net: D6.3 (DIN), D7.1 (DOUT)
- new net: D5.3 (DIN), D6.1 (DOUT)
- new net: D14.3 (DIN), D5.1 (DOUT)
- new net: D13.3 (DIN), D14.1 (DOUT)
- new net: D12.3 (DIN), D13.1 (DOUT)
- new net: D11.3 (DIN), D12.1 (DOUT)
- new net: D10.3 (DIN), D11.1 (DOUT)
- new net: D10.1 (DOUT), D19.3 (DIN)
- new net: D18.3 (DIN), D19.1 (DOUT)
- new net: D17.3 (DIN), D18.1 (DOUT)
- new net: D16.3 (DIN), D17.1 (DOUT)
- new net: D15.3 (DIN), D16.1 (DOUT)
- new net: D15.1 (DOUT), D24.3 (DIN)
- new net: D23.3 (DIN), D24.1 (DOUT)
- new net: D22.3 (DIN), D23.1 (DOUT)
- new net: D21.3 (DIN), D22.1 (DOUT)
- new net: D20.3 (DIN), D21.1 (DOUT)
- new net: D20.1 (DOUT), D29.3 (DIN)
- new net: D28.3 (DIN), D29.1 (DOUT)
- new net: D27.3 (DIN), D28.1 (DOUT)
- new net: D26.3 (DIN), D27.1 (DOUT)
- new net: D25.3 (DIN), D26.1 (DOUT)
- new net: D25.1 (DOUT), D30.3 (DIN)

Commit message: leds
Parts:
- D90: renamed from D0; footprint LED_SMD:LED_SK6812MINI_PLCC4_3.5x3.5mm_P1.75mm -> Custom Footies:sk6812_minie_reversible
- D91: renamed from D1; footprint LED_SMD:LED_SK6812MINI_PLCC4_3.5x3.5mm_P1.75mm -> Custom Footies:sk6812_minie_reversible
- D910: renamed from D10; footprint LED_SMD:LED_SK6812MINI_PLCC4_3.5x3.5mm_P1.75mm -> Custom Footies:sk6812_minie_reversible
- D911: renamed from D11; footprint LED_SMD:LED_SK6812MINI_PLCC4_3.5x3.5mm_P1.75mm -> Custom Footies:sk6812_minie_reversible
- D912: renamed from D12; footprint LED_SMD:LED_SK6812MINI_PLCC4_3.5x3.5mm_P1.75mm -> Custom Footies:sk6812_minie_reversible
- D913: renamed from D13; footprint LED_SMD:LED_SK6812MINI_PLCC4_3.5x3.5mm_P1.75mm -> Custom Footies:sk6812_minie_reversible
- D914: renamed from D14; footprint LED_SMD:LED_SK6812MINI_PLCC4_3.5x3.5mm_P1.75mm -> Custom Footies:sk6812_minie_reversible
- D915: renamed from D15; footprint LED_SMD:LED_SK6812MINI_PLCC4_3.5x3.5mm_P1.75mm -> Custom Footies:sk6812_minie_reversible
- D916: renamed from D16; footprint LED_SMD:LED_SK6812MINI_PLCC4_3.5x3.5mm_P1.75mm -> Custom Footies:sk6812_minie_reversible
- D917: renamed from D17; footprint LED_SMD:LED_SK6812MINI_PLCC4_3.5x3.5mm_P1.75mm -> Custom Footies:sk6812_minie_reversible
- D918: renamed from D18; footprint LED_SMD:LED_SK6812MINI_PLCC4_3.5x3.5mm_P1.75mm -> Custom Footies:sk6812_minie_reversible
- D919: renamed from D19; footprint LED_SMD:LED_SK6812MINI_PLCC4_3.5x3.5mm_P1.75mm -> Custom Footies:sk6812_minie_reversible
- D92: renamed from D2; footprint LED_SMD:LED_SK6812MINI_PLCC4_3.5x3.5mm_P1.75mm -> Custom Footies:sk6812_minie_reversible
- D920: renamed from D20; footprint LED_SMD:LED_SK6812MINI_PLCC4_3.5x3.5mm_P1.75mm -> Custom Footies:sk6812_minie_reversible
- D921: renamed from D21; footprint LED_SMD:LED_SK6812MINI_PLCC4_3.5x3.5mm_P1.75mm -> Custom Footies:sk6812_minie_reversible
- D922: renamed from D22; footprint LED_SMD:LED_SK6812MINI_PLCC4_3.5x3.5mm_P1.75mm -> Custom Footies:sk6812_minie_reversible
- D923: renamed from D23; footprint LED_SMD:LED_SK6812MINI_PLCC4_3.5x3.5mm_P1.75mm -> Custom Footies:sk6812_minie_reversible
- D924: renamed from D24; footprint LED_SMD:LED_SK6812MINI_PLCC4_3.5x3.5mm_P1.75mm -> Custom Footies:sk6812_minie_reversible
- D925: renamed from D25; footprint LED_SMD:LED_SK6812MINI_PLCC4_3.5x3.5mm_P1.75mm -> Custom Footies:sk6812_minie_reversible
- D926: renamed from D26; footprint LED_SMD:LED_SK6812MINI_PLCC4_3.5x3.5mm_P1.75mm -> Custom Footies:sk6812_minie_reversible
- D927: renamed from D27; footprint LED_SMD:LED_SK6812MINI_PLCC4_3.5x3.5mm_P1.75mm -> Custom Footies:sk6812_minie_reversible
- D928: renamed from D28; footprint LED_SMD:LED_SK6812MINI_PLCC4_3.5x3.5mm_P1.75mm -> Custom Footies:sk6812_minie_reversible
- D929: renamed from D29; footprint LED_SMD:LED_SK6812MINI_PLCC4_3.5x3.5mm_P1.75mm -> Custom Footies:sk6812_minie_reversible
- D93: renamed from D3; footprint LED_SMD:LED_SK6812MINI_PLCC4_3.5x3.5mm_P1.75mm -> Custom Footies:sk6812_minie_reversible
- D930: renamed from D30; footprint LED_SMD:LED_SK6812MINI_PLCC4_3.5x3.5mm_P1.75mm -> Custom Footies:sk6812_minie_reversible
- D94: renamed from D4; footprint LED_SMD:LED_SK6812MINI_PLCC4_3.5x3.5mm_P1.75mm -> Custom Footies:sk6812_minie_reversible
- D95: renamed from D5; footprint LED_SMD:LED_SK6812MINI_PLCC4_3.5x3.5mm_P1.75mm -> Custom Footies:sk6812_minie_reversible
- D96: renamed from D6; footprint LED_SMD:LED_SK6812MINI_PLCC4_3.5x3.5mm_P1.75mm -> Custom Footies:sk6812_minie_reversible
- D97: renamed from D7; footprint LED_SMD:LED_SK6812MINI_PLCC4_3.5x3.5mm_P1.75mm -> Custom Footies:sk6812_minie_reversible
- D98: renamed from D8; footprint LED_SMD:LED_SK6812MINI_PLCC4_3.5x3.5mm_P1.75mm -> Custom Footies:sk6812_minie_reversible
- D99: renamed from D9; footprint LED_SMD:LED_SK6812MINI_PLCC4_3.5x3.5mm_P1.75mm -> Custom Footies:sk6812_minie_reversible

Commit message: holes and leds
Parts:
- added U1, U2, U3, U4: HOLE, MountingHole:MountingHole_2.2mm_M2_DIN965_Pad, symbol hole:HOLE
- renumbered U1 to U0
Connections:
- net at D925.1 (DOUT): no longer D930.3 (DIN)
Changed lines of the file:
@@
 COL5
 $Comp
-L promicro:nice_nano U1
+L promicro:nice_nano U0
 U 1 1 5E46BADA
 P 9900 2250
-F 0 "U1" H 9900 3287 60  0000 C CNN
+F 0 "U0" H 9900 3287 60  0000 C CNN
 F 1 "ProMicro" H 9900 3181 60  0000 C CNN
 F 2 "Custom Footies:nice_nano" H 10000 1200 60  0001 C CNN
@@
 Text GLabel 1250 9900 3    50   Input ~ 0
 LED
-Wire Wire Line
-	1250 6900 1900 6900
-Wire Wire Line
-	1900 6900 1900 9900
-Wire Wire Line
-	1900 9900 2500 9900
-Wire Wire Line
-	2500 6900 3150 6900
-Wire Wire Line
-	3150 6900 3150 9900
-Wire Wire Line
-	3150 9900 3800 9900
-Wire Wire Line
-	3800 6900 4450 6900
-Wire Wire Line
-	4450 6900 4450 9900
-Wire Wire Line
-	4450 9900 5050 9900
-Wire Wire Line
-	5050 6900 5750 6900
-Wire Wire Line
-	5750 6900 5750 9900
-Wire Wire Line
-	5750 9900 6350 9900
-Wire Wire Line
-	6350 6900 7000 6900
-Wire Wire Line
-	7000 6900 7000 9900
-Wire Wire Line
-	7000 9900 7650 9900
-Wire Wire Line
-	7650 6900 8350 6900
-Wire Wire Line
-	8350 6900 8350 9900
-Wire Wire Line
-	8350 9900 8900 9900
 Text GLabel 8900 9300 1    50   Input ~ 0
 to_right
 Text GLabel 9250 3400 2    50   Input ~ 0
 to_right
+Wire Wire Line
+	3150 9900 3800 9900
+Wire Wire Line
+	4450 9900 5050 9900
+Wire Wire Line
+	5750 9900 6350 9900
+Wire Wire Line
+	7000 9900 7650 9900
+Wire Wire Line
+	7000 6900 7000 9900
+Wire Wire Line
+	6350 6900 7000 6900
+Wire Wire Line
+	5750 6900 5750 9900
+Wire Wire Line
+	4450 6900 4450 9900
+Wire Wire Line
+	5050 6900 5750 6900
+Wire Wire Line
+	3800 6900 4450 6900
+Wire Wire Line
+	3150 6900 3150 9900
+Wire Wire Line
+	2500 6900 3150 6900
+Wire Wire Line
+	1250 6900 1900 6900
+Wire Wire Line
+	1900 9900 2500 9900
+Wire Wire Line
+	1900 6900 1900 9900
+$Comp
+L hole:HOLE U1
+U 1 1 60668F3F
+P 11150 6550
+F 0 "U1" H 11328 6628 60  0000 L CNN
+F 1 "HOLE" H 11328 6522 60  0000 L CNN
+F 2 "MountingHole:MountingHole_2.2mm_M2_DIN965_Pad" H 11150 6550 60  0001 C CNN
+F 3 "" H 11150 6550 60  0000 C CNN
+	1    11150 6550
+	1    0    0    -1
+$EndComp
+$Comp
+L hole:HOLE U2
+U 1 1 60669CFE
+P 12150 6550
+F 0 "U2" H 12328 6628 60  0000 L CNN
+F 1 "HOLE" H 12328 6522 60  0000 L CNN
+F 2 "MountingHole:MountingHole_2.2mm_M2_DIN965_Pad" H 12150 6550 60  0001 C CNN
+F 3 "" H 12150 6550 60  0000 C CNN
+	1    12150 6550
+	1    0    0    -1
+$EndComp
+$Comp
+L hole:HOLE U3
+U 1 1 6066A776
+P 11150 7200
+F 0 "U3" H 11328 7278 60  0000 L CNN
+F 1 "HOLE" H 11328 7172 60  0000 L CNN
+F 2 "MountingHole:MountingHole_2.2mm_M2_DIN965_Pad" H 11150 7200 60  0001 C CNN
+F 3 "" H 11150 7200 60  0000 C CNN
+	1    11150 7200
+	1    0    0    -1
+$EndComp
+$Comp
+L hole:HOLE U4
+U 1 1 6066B2B8
+P 12200 7200
+F 0 "U4" H 12378 7278 60  0000 L CNN
+F 1 "HOLE" H 12378 7172 60  0000 L CNN
+F 2 "MountingHole:MountingHole_2.2mm_M2_DIN965_Pad" H 12200 7200 60  0001 C CNN
+F 3 "" H 12200 7200 60  0000 C CNN
+	1    12200 7200
+	1    0    0    -1
+$EndComp
 $EndSCHEMATC

Commit message: fin?
Parts:
- added SW91: SW_SPDT, Custom Footies:reversible_power, symbol Switch:SW_SPDT
Connections:
- net B+: now also SW91.2 (B); no longer U0.B+
- new net V+: SW91.1 (A), U0.B+
Other:
- moved on the sheet: J2
Changed lines of the file:
@@
 Text GLabel 9200 1500 0    50   Input ~ 0
 SERIAL
-Text GLabel 10500 1400 2    50   Input ~ 0
-B+
 Text GLabel 9300 1400 0    50   Input ~ 0
 B-
@@
 L Connector:Conn_01x02_Male J2
 U 1 1 60595BC7
-P 9100 4300
-F 0 "J2" H 9208 4481 50  0000 C CNN
-F 1 "battery" H 9208 4390 50  0000 C CNN
-F 2 "Connector_PinSocket_2.54mm:PinSocket_1x02_P2.54mm_Vertical" H 9100 4300 50  0001 C CNN
-F 3 "~" H 9100 4300 50  0001 C CNN
-	1    9100 4300
+P 11850 1650
+F 0 "J2" H 11958 1831 50  0000 C CNN
+F 1 "battery" H 11958 1740 50  0000 C CNN
+F 2 "Connector_PinSocket_2.54mm:PinSocket_1x02_P2.54mm_Vertical" H 11850 1650 50  0001 C CNN
+F 3 "~" H 11850 1650 50  0001 C CNN
+	1    11850 1650
 	1    0    0    -1
 $EndComp
-Text GLabel 9300 4300 2    50   Input ~ 0
-B+
-Text GLabel 9300 4400 2    50   Input ~ 0
+Text GLabel 12050 1750 2    50   Input ~ 0
 B-
 $Comp
@@
 	1    0    0    -1
 $EndComp
+Text GLabel 12250 1200 2    50   Input ~ 0
+B+
+$Comp
+L Switch:SW_SPDT SW91
+U 1 1 60684D01
+P 12050 1200
+F 0 "SW91" H 12050 875 50  0000 C CNN
+F 1 "SW_SPDT" H 12050 966 50  0000 C CNN
+F 2 "Custom Footies:reversible_power" H 12050 1200 50  0001 C CNN
+F 3 "~" H 12050 1200 50  0001 C CNN
+	1    12050 1200
+	-1   0    0    1
+$EndComp
+Text GLabel 12050 1650 2    50   Input ~ 0
+B+
+Text GLabel 11850 1300 0    50   Input ~ 0
+V+
+Text GLabel 10500 1400 2    50   Input ~ 0
+V+
 $EndSCHEMATC

Commit message: moved stuff
Parts:
- added U5: HOLE, MountingHole:MountingHole_2.2mm_M2_DIN965, symbol hole:HOLE
- U1, U2, U3, U4: footprint MountingHole:MountingHole_2.2mm_M2_DIN965_Pad -> MountingHole:MountingHole_2.2mm_M2_DIN965
Other:
- moved on the sheet: U4
Changed lines of the file:
@@
 F 0 "U1" H 11328 6628 60  0000 L CNN
 F 1 "HOLE" H 11328 6522 60  0000 L CNN
-F 2 "MountingHole:MountingHole_2.2mm_M2_DIN965_Pad" H 11150 6550 60  0001 C CNN
+F 2 "MountingHole:MountingHole_2.2mm_M2_DIN965" H 11150 6550 60  0001 C CNN
 F 3 "" H 11150 6550 60  0000 C CNN
 	1    11150 6550
@@
 F 0 "U2" H 12328 6628 60  0000 L CNN
 F 1 "HOLE" H 12328 6522 60  0000 L CNN
-F 2 "MountingHole:MountingHole_2.2mm_M2_DIN965_Pad" H 12150 6550 60  0001 C CNN
+F 2 "MountingHole:MountingHole_2.2mm_M2_DIN965" H 12150 6550 60  0001 C CNN
 F 3 "" H 12150 6550 60  0000 C CNN
 	1    12150 6550
@@
 F 0 "U3" H 11328 7278 60  0000 L CNN
 F 1 "HOLE" H 11328 7172 60  0000 L CNN
-F 2 "MountingHole:MountingHole_2.2mm_M2_DIN965_Pad" H 11150 7200 60  0001 C CNN
+F 2 "MountingHole:MountingHole_2.2mm_M2_DIN965" H 11150 7200 60  0001 C CNN
 F 3 "" H 11150 7200 60  0000 C CNN
 	1    11150 7200
@@
 L hole:HOLE U4
 U 1 1 6066B2B8
-P 12200 7200
-F 0 "U4" H 12378 7278 60  0000 L CNN
-F 1 "HOLE" H 12378 7172 60  0000 L CNN
-F 2 "MountingHole:MountingHole_2.2mm_M2_DIN965_Pad" H 12200 7200 60  0001 C CNN
-F 3 "" H 12200 7200 60  0000 C CNN
-	1    12200 7200
+P 12150 7200
+F 0 "U4" H 12328 7278 60  0000 L CNN
+F 1 "HOLE" H 12328 7172 60  0000 L CNN
+F 2 "MountingHole:MountingHole_2.2mm_M2_DIN965" H 12150 7200 60  0001 C CNN
+F 3 "" H 12150 7200 60  0000 C CNN
+	1    12150 7200
 	1    0    0    -1
 $EndComp
@@
 Text GLabel 10500 1400 2    50   Input ~ 0
 V+
+$Comp
+L hole:HOLE U5
+U 1 1 614B0606
+P 13000 7200
+F 0 "U5" H 13178 7278 60  0000 L CNN
+F 1 "HOLE" H 13178 7172 60  0000 L CNN
+F 2 "MountingHole:MountingHole_2.2mm_M2_DIN965" H 13000 7200 60  0001 C CNN
+F 3 "" H 13000 7200 60  0000 C CNN
+	1    13000 7200
+	1    0    0    -1
+$EndComp
 $EndSCHEMATC
