File: splitreus.kicad_pcb (KiCad board)
At the start: 2 copper layers, 127.5 x 99 mm, 69 parts, among them SW0 SW_PUSH, SW1 SW_PUSH, SW10 SW_PUSH, SW11 SW_PUSH, SW12 SW_PUSH, SW13 SW_PUSH, SW14 SW_PUSH, SW15 SW_PUSH, SW16 SW_PUSH, SW17 SW_PUSH, SW18 SW_PUSH, SW19 SW_PUSH, SW2 SW_PUSH, SW20 SW_PUSH, SW21 SW_PUSH, SW22 SW_PUSH, SW23 SW_PUSH, SW24 SW_PUSH, SW25 SW_PUSH, SW26 SW_PUSH, SW27 SW_PUSH, SW28 SW_PUSH, SW29 SW_PUSH, SW3 SW_PUSH, SW30 SW_PUSH, SW4 SW_PUSH, SW5 SW_PUSH, SW6 SW_PUSH, SW7 SW_PUSH, SW8 SW_PUSH, SW9 SW_PUSH, U1 ProMicro, U2 HOLE, U3 HOLE, U4 HOLE, U5 HOLE, U6 HOLE

Commit message: updates
Parts:
- added JB1: Conn_01x02, Connector_PinSocket_2.54mm:PinSocket_1x02_P2.54mm_Vertical, F.Cu at (107.1, 18.3)
- added U10: HOLE, Custom Footies:breakaway-mousebites, F.Cu at (149.5, 26.4)
- added U11: HOLE, Custom Footies:breakaway-mousebites, F.Cu at (155.5, 24.4)
- added U12: HOLE, Custom Footies:breakaway-mousebites, F.Cu at (149.5, 28.4)
- added U13: HOLE, Custom Footies:breakaway-mousebites, F.Cu at (161.5, 22.4)
- added U14: HOLE, Custom Footies:breakaway-mousebites, F.Cu at (149.5, 30.4)
- added U15: HOLE, Custom Footies:breakaway-mousebites, F.Cu at (155.5, 26.4)
- added U16: HOLE, Custom Footies:breakaway-mousebites, F.Cu at (161.5, 24.4)
- added U17: HOLE, Custom Footies:breakaway-mousebites, F.Cu at (155.5, 28.4)
- added U18: HOLE, Custom Footies:breakaway-mousebites, F.Cu at (155.5, 30.4)
- added U19: HOLE, Custom Footies:breakaway-mousebites, F.Cu at (149.5, 22.4)
- added U20: HOLE, Custom Footies:breakaway-mousebites, F.Cu at (155.5, 32.4)
- added U21: HOLE, Custom Footies:breakaway-mousebites, F.Cu at (161.5, 26.4)
- added U22: HOLE, Custom Footies:breakaway-mousebites, F.Cu at (161.5, 28.4)
- added U23: HOLE, Custom Footies:breakaway-mousebites, F.Cu at (161.5, 30.4)
- added U24: HOLE, Custom Footies:breakaway-mousebites, F.Cu at (161.5, 32.4)
- added U25: HOLE, Custom Footies:breakaway-mousebites_half, F.Cu at (166.3, 22.4)
- added U26: HOLE, Custom Footies:breakaway-mousebites_half, F.Cu at (166.3, 24.4)
- added U27: HOLE, Custom Footies:breakaway-mousebites_half, F.Cu at (166.3, 26.4)
- added U28: HOLE, Custom Footies:breakaway-mousebites_half, F.Cu at (166.3, 28.4)
- added U29: HOLE, Custom Footies:breakaway-mousebites_half, F.Cu at (166.3, 30.4)
- added U7: HOLE, Custom Footies:breakaway-mousebites, F.Cu at (149.5, 32.4)
- added U8: HOLE, Custom Footies:breakaway-mousebites, F.Cu at (149.5, 24.4)
- added U9: HOLE, Custom Footies:breakaway-mousebites, F.Cu at (155.5, 22.4)
- U1: value ProMicro -> nice_nano; footprint keebio:ArduinoProMicro -> Custom Footies:nice_nano
Other:
- outline, holes or cut-outs redrawn

Commit message: design updates
Parts:
- removed JB1: Conn_01x02, Connector_PinSocket_2.54mm:PinSocket_1x02_P2.54mm_Vertical
- removed RST1: RST_SWITCH, Lily58-footprint:TACT_SWITCH_TVBP06
- removed U10, U11, U12, U13, U14, U15, U16, U17, U18, U19, U20, U21, U22, U23, U24, U7, U8, U9: HOLE, Custom Footies:breakaway-mousebites
- removed U25, U26, U27, U28, U29: HOLE, Custom Footies:breakaway-mousebites_half
- removed U4: HOLE, MountingHole:MountingHole_2.5mm
- moved U6 2.02 mm to (81.0, 59.0)
- moved D30 2.00 mm to (114.0, 63.0)
- moved U2 1.03 mm to (27.0, 24.0)
- moved U3 1.03 mm to (27.0, 58.0)
- moved U5 1.03 mm to (81.0, 22.0)
- moved D0 0.75 mm to (0.00, 7.00)
- moved U1 0.65 mm to (108.8, 32.5)
- moved D14 0.65 mm to (36.0, 72.0)
- moved D19 0.65 mm to (54.0, 67.0)
- moved D24 0.65 mm to (72.0, 73.0)
- moved D29 0.65 mm to (90.0, 78.0)
- moved D4 0.65 mm to (0.00, 75.0)
- moved D9 0.65 mm to (18.0, 75.0)
- moved D10 0.65 mm to (36.0, 4.00)
- moved D20 0.65 mm to (72.0, 5.00)
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- renumbered D21 to D1

Commit message: tracies
Parts:
- removed the D1 at (72.0, 22.0)
- removed U6: HOLE, MountingHole:MountingHole_2.5mm
- added D21: 1N4148-F, Custom Footies:smd_diode_reversible, F.Cu at (72.0, 22.0)
- added U4: HOLE, MountingHole:MountingHole_2.5mm, F.Cu at (80.8, 57.5)
Connections:
- U1 pad 1: ROW0 -> (no net)
- U1 pad 10: COL0 -> ROW4
- U1 pad 11: COL1 -> ROW5
- U1 pad 12: COL2 -> COL0
- U1 pad 13: COL3 -> COL1
- U1 pad 14: COL4 -> COL2
- U1 pad 15: COL5 -> COL3
- U1 pad 16: (no net) -> COL4
- U1 pad 17: (no net) -> COL5
- U1 pad 2: ROW1 -> ROW0
- U1 pad 22: RST -> (no net)
- U1 pad 5: ROW2 -> (no net)
- U1 pad 7: ROW3 -> ROW1
- U1 pad 8: ROW4 -> ROW2
- U1 pad 9: ROW5 -> ROW3
Routing:
- net ROW4: track 0.00 -> 319.0 mm, vias 0 -> 1
- net ROW1: track 0.00 -> 296.8 mm
- net ROW0: track 0.00 -> 279.5 mm
- net COL0: track 0.00 -> 252.3 mm, vias 0 -> 3
- net COL5: track 0.00 -> 248.4 mm, vias 0 -> 1
- net COL1: track 0.00 -> 224.9 mm, vias 0 -> 3
- net ROW2: track 0.00 -> 223.0 mm, vias 0 -> 3
- net ROW3: track 0.00 -> 210.4 mm, vias 0 -> 3
- net COL3: track 0.00 -> 200.1 mm, vias 0 -> 2
- net COL2: track 0.00 -> 187.1 mm, vias 0 -> 4
- net COL4: track 0.00 -> 175.1 mm, vias 0 -> 3
- net Net-(D21-Pad1): track 0.00 -> 31.5 mm, vias 0 -> 1
- net Net-(D8-Pad1): track 0.00 -> 31.1 mm, vias 0 -> 1
- net Net-(D18-Pad1): track 0.00 -> 31.1 mm, vias 0 -> 1
- net Net-(D6-Pad1): track 0.00 -> 31.1 mm, vias 0 -> 1
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Other:
- outline, holes or cut-outs redrawn

Commit message: aa
Parts:
- added SW91: SW_PUSH, Lily58-footprint:TACT_SWITCH_TVBP06, F.Cu at (113.0, 49.8)
Connections:
- U1 pad 22: (no net) -> RST
Routing:
- net GND: track 18.8 -> 59.3 mm, vias 0 -> 1
- net RST: track 0.00 -> 27.2 mm
- net COL5: track 248.4 -> 249.5 mm, vias 1 -> 2
- net COL4: track 175.1 -> 175.7 mm
Changed lines of the file:
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@@
     (thickness 1.6)
     (drawings 459)
-    (tracks 1086)
+    (tracks 1106)
     (zones 0)
-    (modules 67)
-    (nets 45)
+    (modules 68)
+    (nets 46)
   )
   (page A4)
@@
   (net 43 COL1)
   (net 44 "Net-(D20-Pad1)")
+  (net 45 RST)
   (net_class Default "This is the default net class."
     (clearance 0.2)
@@
     (add_net ROW4)
     (add_net ROW5)
+    (add_net RST)
+  )
+  (module Lily58-footprint:TACT_SWITCH_TVBP06 (layer F.Cu)
+    (at 113.048 49.828 180)
+    (fp_text reference SW91 (at 0 -1.7) (layer F.SilkS) hide
+      (effects (font (size 1 1) (thickness 0.15)))
+    )
+    (fp_text value SW_PUSH (at 0 2) (layer F.Fab) hide
+      (effects (font (size 1 1) (thickness 0.15)))
+    )
+    (fp_line (start -3 -1.8) (end -3 -1.1) (layer B.SilkS) (width 0.15))
+    (fp_line (start -3 1.7) (end -3 1.1) (layer B.SilkS) (width 0.15))
+    (fp_line (start 3 1.7) (end 3 1.1) (layer B.SilkS) (width 0.15))
+    (fp_line (start 3 -1.8) (end 3 -1.1) (layer B.SilkS) (width 0.15))
+    (fp_line (start -3 -1.8) (end -3 -1.1) (layer F.SilkS) (width 0.15))
+    (fp_line (start -3 1.7) (end -3 1.1) (layer F.SilkS) (width 0.15))
+    (fp_line (start 3 1.7) (end 3 1.1) (layer F.SilkS) (width 0.15))
+    (fp_line (start 3 -1.8) (end 3 -1.1) (layer F.SilkS) (width 0.15))
+    (fp_line (start -3 1.7) (end 3 1.7) (layer F.SilkS) (width 0.15))
+    (fp_line (start 3 -1.8) (end -3 -1.8) (layer F.SilkS) (width 0.15))
+    (fp_line (start 3 1.7) (end -3 1.7) (layer B.SilkS) (width 0.15))
+    (fp_line (start -3 -1.8) (end 3 -1.8) (layer B.SilkS) (width 0.15))
+    (fp_line (start -3 -1.8) (end 2.9 -1.8) (layer B.SilkS) (width 0.15))
+    (fp_text user RESET (at 0 0) (layer B.SilkS)
+      (effects (font (size 0.8 0.8) (thickness 0.15)) (justify mirror))
+    )
+    (fp_text user RESET (at 0 0 180) (layer F.SilkS)
+      (effects (font (size 0.8 0.8) (thickness 0.15)))
+    )
+    (pad 2 thru_hole circle (at 3.25 0 180) (size 2 2) (drill 1.3) (layers *.Cu *.Mask)
+      (net 38 GND))
+    (pad 1 thru_hole circle (at -3.25 0 180) (size 2 2) (drill 1.3) (layers *.Cu *.Mask)
+      (net 45 RST))
   )
   (module MountingHole:MountingHole_2.5mm (layer F.Cu)
@@
     (pad 23 thru_hole circle (at -11.43 -7.62 270) (size 1.7526 1.7526) (drill 1.0922) (layers *.Cu *.SilkS *.Mask)
       (net 38 GND))
-    (pad 22 thru_hole circle (at -8.89 -7.62 270) (size 1.7526 1.7526) (drill 1.0922) (layers *.Cu *.SilkS *.Mask))
+    (pad 22 thru_hole circle (at -8.89 -7.62 270) (size 1.7526 1.7526) (drill 1.0922) (layers *.Cu *.SilkS *.Mask)
+      (net 45 RST))
     (pad 21 thru_hole circle (at -6.35 -7.62 270) (size 1.7526 1.7526) (drill 1.0922) (layers *.Cu *.SilkS *.Mask))
     (pad 20 thru_hole circle (at -3.81 -7.62 270) (size 1.7526 1.7526) (drill 1.0922) (layers *.Cu *.SilkS *.Mask))
@@
   (segment (start 113.848 23.628) (end 116.388 21.088) (width 0.25) (layer F.Cu) (net 38))
   (segment (start 101.148 23.628) (end 101.148 26.168) (width 0.25) (layer F.Cu) (net 38))
+  (segment (start 114.597275 38.378) (end 114.597275 52.057275) (width 0.25) (layer B.Cu) (net 38))
+  (segment (start 101.148 26.168) (end 102.387275 26.168) (width 0.25) (layer B.Cu) (net 38))
+  (segment (start 102.387275 26.168) (end 114.597275 38.378) (width 0.25) (layer B.Cu) (net 38))
+  (segment (start 114.597275 52.057275) (end 115.388 52.848) (width 0.25) (layer B.Cu) (net 38))
+  (segment (start 115.388 52.848) (end 115.388 52.848) (width 0.25) (layer B.Cu) (net 38))
+  (via (at 115.388 52.848) (size 0.8) (drill 0.4) (layers F.Cu B.Cu) (net 38))
+  (segment (start 110.797999 50.827999) (end 109.798 49.828) (width 0.25) (layer F.Cu) (net 38))
+  (segment (start 113.217999 53.247999) (end 110.797999 50.827999) (width 0.25) (layer F.Cu) (net 38))
+  (segment (start 115.388 52.848) (end 114.988001 53.247999) (width 0.25) (layer F.Cu) (net 38))
+  (segment (start 114.988001 53.247999) (end 113.217999 53.247999) (width 0.25) (layer F.Cu) (net 38))
   (segment (start 73.7 39) (end 74.6253 39) (width 0.25) (layer B.Cu) (net 39))
   (segment (start 73.7 38.4873) (end 74.107 38.4873) (width 0.25) (layer F.Cu) (net 39))
@@
   (segment (start 78.8302 33.5461) (end 78.1286 33.5461) (width 0.25) (layer F.Cu) (net 39))
   (segment (start 78.1286 33.5461) (end 73.7 37.9747) (width 0.25) (layer F.Cu) (net 39))
-  (segment (start 116.388 38.868) (end 115.118 37.598) (width 0.25) (layer F.Cu) (net 39))
-  (segment (start 115.118 37.598) (end 98.3709 37.598) (width 0.25) (layer F.Cu) (net 39))
   (segment (start 98.3709 37.598) (end 96.5262 35.7533) (width 0.25) (layer F.Cu) (net 39))
   (segment (start 96.5262 35.7533) (end 91.9843 35.7533) (width 0.25) (layer F.Cu) (net 39))
@@
   (via (at 74.2137 20.4987) (size 0.8) (layers F.Cu B.Cu) (net 39))
   (via (at 73.7 54.6096) (size 0.8) (layers F.Cu B.Cu) (net 39))
+  (segment (start 101.655926 37.598) (end 98.3709 37.598) (width 0.25) (layer F.Cu) (net 39))
+  (segment (start 103.663827 39.605901) (end 101.655926 37.598) (width 0.25) (layer F.Cu) (net 39))
+  (segment (start 114.410824 39.605901) (end 103.663827 39.605901) (width 0.25) (layer F.Cu) (net 39))
+  (segment (start 116.388 38.868) (end 115.148725 38.868) (width 0.25) (layer F.Cu) (net 39))
+  (segment (start 115.148725 38.868) (end 114.410824 39.605901) (width 0.25) (layer F.Cu) (net 39))
   (segment (start 116.388 43.948) (end 115.118 42.678) (width 0.25) (layer F.Cu) (net 40))
   (segment (start 115.118 42.678) (end 100.1001 42.678) (width 0.25) (layer F.Cu) (net 40))
@@
   (segment (start 91.7 26.4873) (end 91.7 27) (width 0.25) (layer B.Cu) (net 41))
   (segment (start 91.7 44) (end 92.6253 44) (width 0.25) (layer B.Cu) (net 41))
-  (segment (start 114 38.8809) (end 102.8979 38.8809) (width 0.25) (layer B.Cu) (net 41))
+  (segment (start 114 38.8809) (end 112.8251 38.8809) (width 0.25) (layer B.Cu) (net 41))
   (segment (start 102.8979 38.8809) (end 102.8979 38.8808) (width 0.25) (layer B.Cu) (net 41))
   (segment (start 102.8979 38.8808) (end 101.6407 40.138) (width 0.25) (layer B.Cu) (net 41))
@@
   (segment (start 91.7 26.4873) (end 91.7 25.9747) (width 0.25) (layer B.Cu) (net 41))
   (segment (start 114 38.8809) (end 114 61.3) (width 0.25) (layer B.Cu) (net 41))
-  (segment (start 116.388 36.328) (end 114 38.716) (width 0.25) (layer B.Cu) (net 41))
-  (segment (start 114 38.716) (end 114 38.8809) (width 0.25) (layer B.Cu) (net 41))
   (segment (start 91.7 61.5562) (end 91.7 62.0253) (width 0.25) (layer B.Cu) (net 41))
   (segment (start 91.7 61) (end 91.7 61.5562) (width 0.25) (layer B.Cu) (net 41))
@@
   (segment (start 114 61.3) (end 114 60.3747) (width 0.25) (layer F.Cu) (net 41))
   (via (at 92.9791 44.1975) (size 0.8) (layers F.Cu B.Cu) (net 41))
+  (segment (start 112.8251 38.8809) (end 102.8979 38.8809) (width 0.25) (layer B.Cu) (net 41))
+  (via (at 112.8251 38.8809) (size 0.8) (drill 0.4) (layers F.Cu B.Cu) (net 41))
+  (segment (start 113.8351 38.8809) (end 116.388 36.328) (width 0.25) (layer F.Cu) (net 41))
+  (segment (start 112.8251 38.8809) (end 113.8351 38.8809) (width 0.25) (layer F.Cu) (net 41))
   (segment (start 55.7 -1) (end 56.6253 -1) (width 0.25) (layer F.Cu) (net 42))
   (segment (start 57.3459 16) (end 55.7 16) (width 0.25) (layer F.Cu) (net 42))
@@
   (segment (start 70.3 5) (end 70.3 3.9747) (width 0.25) (layer F.Cu) (net 44))
   (via (at 70.7506 3.6764) (size 0.8) (layers F.Cu B.Cu) (net 44))
+  (segment (start 115.511701 24.504299) (end 116.388 23.628) (width 0.25) (layer B.Cu) (net 45))
+  (segment (start 115.186699 24.829301) (end 115.511701 24.504299) (width 0.25) (layer B.Cu) (net 45))
+  (segment (start 115.186699 47.302486) (end 115.186699 24.829301) (width 0.25) (layer B.Cu) (net 45))
+  (segment (start 116.298 49.828) (end 116.298 48.413787) (width 0.25) (layer B.Cu) (net 45))
+  (segment (start 116.298 48.413787) (end 115.186699 47.302486) (width 0.25) (layer B.Cu) (net 45))
 )

Commit message: upload
Parts:
- removed D0, D1, D10, D15, D2, D20, D25, D3, D4, D5: 1N4148-F, Custom Footies:smd_diode_reversible
- removed SW0, SW1, SW10, SW15, SW2, SW20, SW25, SW3, SW4, SW5: SW_PUSH, daprice_kail_mx:Kailh_socket_PG1350_reversible
Routing:
- net ROW0: track 279.5 -> 0.00 mm
- net COL0: track 252.3 -> 131.4 mm, vias 3 -> 0
- net ROW1: track 296.8 -> 202.2 mm
- net Net-(D5-Pad1): track 31.1 -> 0.00 mm, vias 1 -> 0
- net Net-(D3-Pad1): track 31.1 -> 0.00 mm, vias 1 -> 0
- net Net-(D4-Pad1): track 31.1 -> 0.00 mm, vias 1 -> 0
- net Net-(D0-Pad1): track 31.1 -> 0.00 mm, vias 1 -> 0
- net Net-(D15-Pad1): track 31.1 -> 0.00 mm, vias 1 -> 0
- net Net-(D25-Pad1): track 30.3 -> 0.00 mm, vias 1 -> 0
- net Net-(D20-Pad1): track 29.2 -> 0.00 mm, vias 1 -> 0
- net Net-(D2-Pad1): track 29.1 -> 0.00 mm, vias 1 -> 0
- net Net-(D10-Pad1): track 28.6 -> 0.00 mm, vias 1 -> 0
- net Net-(D1-Pad1): track 28.6 -> 0.00 mm, vias 1 -> 0
- net ROW2: track 223.0 -> 201.2 mm
- net COL4: track 175.7 -> 154.2 mm
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Other:
- board size 127.5 x 99 mm -> 109.5 x 82 mm

Commit message: changes
Parts:
- added J3: Conn_01x04, Connector:FanPinHeader_1x04_P2.54mm_Vertical, F.Cu at (125.5, 44.4)
- moved SW91 42.0 mm to (96.2, 11.3), turned to 0 degrees
Connections:
- U1 pad 12: COL0 -> (no net)
- U1 pad 2: ROW0 -> (no net)
- U1 pad 21: (no net) -> VCC
- U1 pad 5: (no net) -> SCL
- U1 pad 6: (no net) -> SDA
Routing:
- net ROW4: track 304.9 -> 0.00 mm, vias 1 -> 0
- net COL5: track 249.5 -> 0.00 mm, vias 2 -> 0
- net COL1: track 220.2 -> 0.00 mm, vias 2 -> 0
- net ROW1: track 202.2 -> 0.00 mm
- net ROW2: track 201.2 -> 0.00 mm, vias 3 -> 0
- net COL3: track 198.1 -> 0.00 mm, vias 2 -> 0
- net ROW3: track 195.9 -> 0.00 mm, vias 3 -> 0
- net COL2: track 184.7 -> 0.00 mm, vias 4 -> 0
- net COL4: track 154.2 -> 0.00 mm, vias 3 -> 0
- net COL0: track 131.4 -> 0.00 mm
- net GND: track 59.3 -> 0.00 mm, vias 1 -> 0
- net Net-(D21-Pad1): track 31.5 -> 0.00 mm, vias 1 -> 0
- net Net-(D8-Pad1): track 31.1 -> 0.00 mm, vias 1 -> 0
- net Net-(D18-Pad1): track 31.1 -> 0.00 mm, vias 1 -> 0
- net Net-(D6-Pad1): track 31.1 -> 0.00 mm, vias 1 -> 0
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
Commit message: changes
Parts:
- removed J3: Conn_01x04, Connector:FanPinHeader_1x04_P2.54mm_Vertical
- moved U1 0.49 mm to (108.8, 32.0)
Changed lines of the file:
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@@
     (tracks 0)
     (zones 0)
-    (modules 49)
+    (modules 48)
     (nets 37)
   )
@@
     (uvia_dia 0.3)
     (uvia_drill 0.1)
+    (add_net COL0)
     (add_net COL1)
     (add_net COL2)
@@
     (add_net VCC)
   )
-  (module Connector:FanPinHeader_1x04_P2.54mm_Vertical (layer F.Cu)
-    (at 125.518 44.368 90)
-    (descr "4-pin CPU fan Through hole pin header, e.g. for Wieson part number 2366C888-007 Molex 47053-1000, Foxconn HF27040-M1, Tyco 1470947-1 or equivalent, see http://www.formfactors.org/developer%5Cspecs%5Crev1_2_public.pdf")
-    (tags "pin header 4-pin CPU fan")
-    (fp_text reference J3 (at 4 -3.55 90) (layer F.SilkS)
-      (effects (font (size 1 1) (thickness 0.15)))
-    )
-    (fp_text value Conn_01x04 (at 4.05 4.35 90) (layer F.Fab)
-      (effects (font (size 1 1) (thickness 0.15)))
-    )
-    (fp_line (start 9.35 -3.2) (end 9.35 3.8) (layer F.CrtYd) (width 0.05))
-    (fp_line (start 9.35 -3.2) (end -1.75 -3.2) (layer F.CrtYd) (width 0.05))
-    (fp_line (start -1.75 3.8) (end 9.35 3.8) (layer F.CrtYd) (width 0.05))
-    (fp_line (start -1.75 3.8) (end -1.75 -3.2) (layer F.CrtYd) (width 0.05))
-    (fp_line (start 5.08 2.29) (end 5.08 3.3) (layer F.SilkS) (width 0.12))
-    (fp_line (start 0 2.29) (end 5.08 2.29) (layer F.SilkS) (width 0.12))
-    (fp_line (start 0 3.3) (end 0 2.29) (layer F.SilkS) (width 0.12))
-    (fp_line (start -1.25 -2.5) (end 4.4 -2.5) (layer F.Fab) (width 0.1))
-    (fp_line (start -1.25 3.3) (end -1.25 -2.5) (layer F.Fab) (width 0.1))
-    (fp_line (start -1.2 3.3) (end -1.25 3.3) (layer F.Fab) (width 0.1))
-    (fp_line (start 8.85 3.3) (end -1.2 3.3) (layer F.Fab) (width 0.1))
-    (fp_line (start 8.85 -2.5) (end 8.85 3.3) (layer F.Fab) (width 0.1))
-    (fp_line (start 5.75 -2.5) (end 8.85 -2.5) (layer F.Fab) (width 0.1))
-    (fp_line (start 0 2.3) (end 0 3.3) (layer F.Fab) (width 0.1))
-    (fp_line (start 5.1 2.3) (end 0 2.3) (layer F.Fab) (width 0.1))
-    (fp_line (start 5.1 3.3) (end 5.1 2.3) (layer F.Fab) (width 0.1))
-    (fp_line (start -1.35 3.4) (end -1.35 -2.6) (layer F.SilkS) (width 0.12))
-    (fp_line (start 8.95 3.4) (end -1.35 3.4) (layer F.SilkS) (width 0.12))
-    (fp_line (start 8.95 -2.55) (end 8.95 3.4) (layer F.SilkS) (width 0.12))
-    (fp_line (start 5.75 -2.55) (end 8.95 -2.55) (layer F.SilkS) (width 0.12))
-    (fp_line (start -1.35 -2.6) (end 4.4 -2.6) (layer F.SilkS) (width 0.12))
-    (fp_text user %R (at 1.85 -1.75 90) (layer F.Fab)
-      (effects (font (size 1 1) (thickness 0.15)))
-    )
-    (pad "" np_thru_hole circle (at 5.08 -2.16 180) (size 1.1 1.1) (drill 1.1) (layers *.Cu *.Mask))
-    (pad 4 thru_hole oval (at 7.62 0 180) (size 2.03 1.73) (drill 1.02) (layers *.Cu *.Mask)
-      (net 27 GND))
-    (pad 3 thru_hole oval (at 5.08 0 180) (size 2.03 1.73) (drill 1.02) (layers *.Cu *.Mask)
-      (net 34 VCC))
-    (pad 2 thru_hole oval (at 2.54 0 180) (size 2.03 1.73) (drill 1.02) (layers *.Cu *.Mask)
-      (net 35 SDA))
-    (pad 1 thru_hole rect (at 0 0 180) (size 2.03 1.73) (drill 1.02) (layers *.Cu *.Mask)
-      (net 36 SCL))
-    (model ${KISYS3DMOD}/Connector.3dshapes/FanPinHeader_1x04_P2.54mm_Vertical.wrl
-      (at (xyz 0 0 0))
-      (scale (xyz 1 1 1))
-      (rotate (xyz 0 0 0))
-    )
-  )
   (module Lily58-footprint:TACT_SWITCH_TVBP06 (layer F.Cu)
     (at 96.218 11.298)
@@
   )
   (module "Custom Footies:nice_nano" (layer F.Cu)
-    (at 108.768 32.518 270)
+    (at 108.768 32.028 270)
     (fp_text reference U1 (at 0 1.625 90) (layer F.SilkS) hide
       (effects (font (size 1.27 1.524) (thickness 0.2032)))

Commit message: change
Parts:
- added J3: Conn_01x04, Connector:FanPinHeader_1x04_P2.54mm_Vertical, F.Cu at (112.3, 49.0)
- added U6: HOLE, MountingHole:MountingHole_2.2mm_M2, F.Cu at (26.7, 6.95)
- added U7: HOLE, MountingHole:MountingHole_2.2mm_M2, F.Cu at (150.2, 28.1)
- added U8: HOLE, MountingHole:MountingHole_2.2mm_M2, F.Cu at (115.2, 53.9)
- added U9: HOLE, MountingHole:MountingHole_2.2mm_M2, F.Cu at (98.1, 12.1)
- U2, U3, U4, U5: footprint MountingHole:MountingHole_2.5mm -> MountingHole:MountingHole_2.2mm_M2
- moved SW91 63.6 mm to (98.9, 74.8), turned to 90 degrees
- moved U2 25.5 mm to (9.38, 42.5)
- moved U4 22.6 mm to (62.2, 70.4)
- moved U5 21.9 mm to (66.3, 5.71)
- moved U3 16.0 mm to (27.4, 74.0)
