File: pro_micro_adapter/pma/pma.kicad_pcb (KiCad board)
At the start: 2 copper layers, 16 x 38 mm, 4 parts, among them J1 Lily58-cache_MJ-4PP-9, J2 4PIN, J3 4PIN, U1 ProMicro

Commit message: silk
Parts:
- removed J3: 4PIN, Connector_PinHeader_2.54mm:PinHeader_1x04_P2.54mm_Vertical
- J1: footprint Custom Footies:PJ-606-6A -> Lily58-footprint:MJ-4PP-9
- J2: footprint Connector_PinHeader_2.54mm:PinHeader_1x04_P2.54mm_Vertical -> Custom Footies:PinHeader_1x04_P2.54mm_REVERSIBLE
- moved J1 15.5 mm to (8.40, -1.66), turned to 270 degrees
- moved J2 1.85 mm to (4.94, 19.5)
Connections:
- J1 pad 1: (no net) -> Net-(J1-Pad1)
- J2 pad 1: SDA -> GND
- J2 pad 2: SCL -> VCC
- J2 pad 3: VCC -> SCL
- J2 pad 4: GND -> SDA
Routing:
- net GND: track 0.00 -> 69.9 mm
- net VCC: track 0.00 -> 47.1 mm
- net SDA: track 0.00 -> 34.6 mm
- net SCL: track 0.00 -> 29.5 mm
- net SERIAL: track 0.00 -> 19.8 mm
- net Net-(J1-Pad1): track 0.00 -> 5.95 mm
- added copper zone on B.Cu, net (none)
- added copper zone on F.Cu, net (none)
